File: Barómetro DPS310.kicad_sch (KiCad schematic)
At the start: 6 parts, among them U5 DPS310XTSA1

Commit message: Cantidad de errores en la PCB: 29
Parts:
- C24, C25: footprint easyeda2kicad:C0402 -> ARLISS-footprints:C0402
- U5: footprint easyeda2kicad:LGA-8_DPS310XTSA1 -> ARLISS-footprints:LGA-8_DPS310XTSA1
Changed lines of the file:
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@@
 			)
 		)
-		(property "Footprint" "easyeda2kicad:C0402"
+		(property "Footprint" "ARLISS-footprints:C0402"
 			(at 210.82 100.33 0)
 			(hide yes)
@@
 			)
 		)
-		(property "Footprint" "easyeda2kicad:LGA-8_DPS310XTSA1"
+		(property "Footprint" "ARLISS-footprints:LGA-8_DPS310XTSA1"
 			(at 166.37 105.41 0)
 			(hide yes)
@@
 			)
 		)
-		(property "Footprint" "easyeda2kicad:C0402"
+		(property "Footprint" "ARLISS-footprints:C0402"
 			(at 191.77 81.28 0)
 			(hide yes)

Commit message: Cantidad de errores de la placa: 05
Parts:
- R4, R5: footprint easyeda2kicad:R0603 -> ARLISS-footprints:R0603
Changed lines of the file:
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@@
 			)
 		)
-		(property "Footprint" "easyeda2kicad:R0603"
+		(property "Footprint" "ARLISS-footprints:R0603"
 			(at 142.24 88.9 0)
 			(hide yes)
@@
 			)
 		)
-		(property "Footprint" "easyeda2kicad:R0603"
+		(property "Footprint" "ARLISS-footprints:R0603"
 			(at 151.13 87.63 0)
 			(hide yes)

Commit message: Cantidad de errores en la placa: 04
Parts:
- R1: footprint (none) -> ARLISS-footprints:R0603; LCSC Part (none) -> C5552302
Changed lines of the file:
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@@
 			)
 		)
-		(property "Footprint" ""
+		(property "Footprint" "ARLISS-footprints:R0603"
 			(at 179.832 105.41 90)
 			(hide yes)
@@
 			)
 		)
-		(property "Datasheet" ""
+		(property "Datasheet" "https://www.lcsc.com/datasheet/C5552302.pdf?spm=wm.sxq.pdf.fd___wm.fly.bg.1.cbh&lcsc_vid=FVBZXlJVElFWAVdTTgAPVAcHR1hXAlIFT1cMUAFWQVYxVlNeRlVfVFdeR1NaXzsOAxUeFF5JWBYZEEoKFBINSQcJGk4dAgUUFAk%3D"
 			(at 181.61 105.41 0)
 			(hide yes)
@@
 			(at 181.61 105.41 0)
 			(hide yes)
+			(show_name no)
+			(do_not_autoplace no)
+			(effects
+				(font
+					(size 1.27 1.27)
+				)
+			)
+		)
+		(property "LCSC Part" "C5552302"
+			(at 181.61 105.41 0)
+			(hide yes)

Commit message: PCB ordenada V1
Parts:
- removed R4, R5: 4.7K, ARLISS-footprints:R0603, symbol CANSAT_STM32_symbols:RC0603FR-074K7L

Commit message: Primer Ruteo de PCB
Parts:
- C24, C25: footprint ARLISS-footprints:C0402 -> Capacitor_SMD:C_0402_1005Metric_Pad0.74x0.62mm_HandSolder
Changed lines of the file:
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@@
 			)
 		)
-		(property "Footprint" "ARLISS-footprints:C0402"
+		(property "Footprint" "Capacitor_SMD:C_0402_1005Metric_Pad0.74x0.62mm_HandSolder"
 			(at 210.82 100.33 0)
 			(hide yes)
@@
 			)
 		)
-		(property "Footprint" "ARLISS-footprints:C0402"
+		(property "Footprint" "Capacitor_SMD:C_0402_1005Metric_Pad0.74x0.62mm_HandSolder"
 			(at 191.77 81.28 0)
 			(hide yes)

Commit message: Arreglos de esquemático
Parts:
- R1: footprint ARLISS-footprints:R0603 -> Resistor_SMD:R_0603_1608Metric_Pad0.98x0.95mm_HandSolder
Changed lines of the file:
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@@
 			)
 		)
-		(property "Footprint" "ARLISS-footprints:R0603"
+		(property "Footprint" "Resistor_SMD:R_0603_1608Metric_Pad0.98x0.95mm_HandSolder"
 			(at 179.832 105.41 90)
 			(hide yes)

Commit message: Arreglando footprints
Parts:
- C27: renamed from C24; footprint Capacitor_SMD:C_0402_1005Metric_Pad0.74x0.62mm_HandSolder -> Capacitor_SMD:C_0603_1608Metric_Pad1.08x0.95mm_HandSolder; Manufacturer CCTC(三环) -> (none)
- C28: renamed from C25; footprint Capacitor_SMD:C_0402_1005Metric_Pad0.74x0.62mm_HandSolder -> Capacitor_SMD:C_0603_1608Metric_Pad1.08x0.95mm_HandSolder; Manufacturer CCTC(三环) -> (none)
- U5: Manufacturer Infineon(英飞凌) -> (none)
- renumbered R1 to R11
Other:
- company: (none) -> TOMEK TEAM
Changed lines of the file:
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@@
 	(generator_version "10.0")
 	(paper "A4")
+	(title_block
+		(company "TOMEK TEAM")
+	)
 	(junction
 		(at 184.15 90.17)
@@
 		(in_pos_files yes)
 		(dnp no)
-		(property "Reference" "#PWR054"
+		(property "Reference" "#PWR063"
 			(at 146.05 90.17 0)
 			(hide yes)
@@
 			(project "ARLISS_STM32_2026"
 				(path "/9719ea46-14c4-4409-9c57-49dd5454c03f/9e299f07-4887-409a-8623-587b30453872"
-					(reference "#PWR054")
+					(reference "#PWR063")
 					(unit 1)
 				)
@@
 		(dnp no)
 		(fields_autoplaced yes)
-		(property "Reference" "#PWR060"
+		(property "Reference" "#PWR065"
 			(at 181.61 118.11 0)
 			(hide yes)
@@
 			(project "ARLISS_STM32_2026"
 				(path "/9719ea46-14c4-4409-9c57-49dd5454c03f/9e299f07-4887-409a-8623-587b30453872"
-					(reference "#PWR060")
+					(reference "#PWR065")
 					(unit 1)
 				)
@@
 		(dnp no)
 		(fields_autoplaced yes)
-		(property "Reference" "#PWR058"
+		(property "Reference" "#PWR068"
 			(at 203.2 114.3 0)
 			(hide yes)
@@
 			(project "ARLISS_STM32_2026"
 				(path "/9719ea46-14c4-4409-9c57-49dd5454c03f/9e299f07-4887-409a-8623-587b30453872"
-					(reference "#PWR058")
+					(reference "#PWR068")
 					(unit 1)
 				)
@@
 		(dnp no)
 		(fields_autoplaced yes)
-		(property "Reference" "R1"
+		(property "Reference" "R11"
 			(at 184.15 104.1399 0)
 			(show_name no)
@@
 			(project "ARLISS_STM32_2026"
 				(path "/9719ea46-14c4-4409-9c57-49dd5454c03f/9e299f07-4887-409a-8623-587b30453872"
-					(reference "R1")
+					(reference "R11")
 					(unit 1)
 				)
@@
 		(dnp no)
 		(fields_autoplaced yes)
-		(property "Reference" "#PWR055"
+		(property "Reference" "#PWR067"
 			(at 198.12 93.98 0)
 			(hide yes)
@@
 			(project "ARLISS_STM32_2026"
 				(path "/9719ea46-14c4-4409-9c57-49dd5454c03f/9e299f07-4887-409a-8623-587b30453872"
-					(reference "#PWR055")
+					(reference "#PWR067")
 					(unit 1)
 				)
@@
 		(dnp no)
 		(fields_autoplaced yes)
-		(property "Reference" "#PWR056"
+		(property "Reference" "#PWR066"
 			(at 184.15 68.58 0)
 			(hide yes)
@@
 			(project "ARLISS_STM32_2026"
 				(path "/9719ea46-14c4-4409-9c57-49dd5454c03f/9e299f07-4887-409a-8623-587b30453872"
-					(reference "#PWR056")
+					(reference "#PWR066")
 					(unit 1)
 				)
@@
 		(dnp no)
 		(fields_autoplaced yes)
-		(property "Reference" "C25"
+		(property "Reference" "C28"
 			(at 207.01 99.0599 90)
 			(show_name no)
@@
 			)
 		)
-		(property "Footprint" "Capacitor_SMD:C_0402_1005Metric_Pad0.74x0.62mm_HandSolder"
+		(property "Footprint" "Capacitor_SMD:C_0603_1608Metric_Pad1.08x0.95mm_HandSolder"
 			(at 210.82 100.33 0)
 			(hide yes)
@@
 			)
 		)
-		(property "Manufacturer" "CCTC(三环)"
-			(at 215.9 100.33 0)
-			(hide yes)
-			(show_name no)
-			(do_not_autoplace no)
-			(effects
-				(font
-					(size 1.27 1.27)
-				)
-			)
-		)
 		(property "MPN" "TCC0402X7R104J500AT"
 			(at 218.44 100.33 0)
@@
 			(project "ARLISS_STM32_2026"
 				(path "/9719ea46-14c4-4409-9c57-49dd5454c03f/9e299f07-4887-409a-8623-587b30453872"
-					(reference "C25")
+					(reference "C28")
 					(unit 1)
 				)
@@
 		(dnp no)
 		(fields_autoplaced yes)
-		(property "Reference" "#PWR057"
+		(property "Reference" "#PWR069"
 			(at 203.2 95.25 0)
 			(hide yes)
@@
 			(project "ARLISS_STM32_2026"
 				(path "/9719ea46-14c4-4409-9c57-49dd5454c03f/9e299f07-4887-409a-8623-587b30453872"
-					(reference "#PWR057")
+					(reference "#PWR069")
 					(unit 1)
 				)
@@
 			)
 		)
-		(property "Manufacturer" "Infineon(英飞凌)"
-			(at 166.37 110.49 0)
-			(hide yes)
-			(show_name no)
-			(do_not_autoplace no)
-			(effects
-				(font
-					(size 1.27 1.27)
-				)
-			)
-		)
 		(property "MPN" "DPS310"
 			(at 166.37 113.03 0)
@@
 		(dnp no)
 		(fields_autoplaced yes)
-		(property "Reference" "#PWR053"
+		(property "Reference" "#PWR064"
 			(at 186.69 92.71 0)
 			(hide yes)
@@
 			(project "ARLISS_STM32_2026"
 				(path "/9719ea46-14c4-4409-9c57-49dd5454c03f/9e299f07-4887-409a-8623-587b30453872"
-					(reference "#PWR053")
+					(reference "#PWR064")
 					(unit 1)
 				)
@@
 		(dnp no)
 		(fields_autoplaced yes)
-		(property "Reference" "C24"
+		(property "Reference" "C27"
 			(at 187.96 80.0099 90)
 			(show_name no)
@@
 			)
 		)
-		(property "Footprint" "Capacitor_SMD:C_0402_1005Metric_Pad0.74x0.62mm_HandSolder"
+		(property "Footprint" "Capacitor_SMD:C_0603_1608Metric_Pad1.08x0.95mm_HandSolder"
 			(at 191.77 81.28 0)
 			(hide yes)
@@
 			)
 		)
-		(property "Manufacturer" "CCTC(三环)"
-			(at 196.85 81.28 0)
-			(hide yes)
-			(show_name no)
-			(do_not_autoplace no)
-			(effects
-				(font
-					(size 1.27 1.27)
-				)
-			)
-		)
 		(property "MPN" "TCC0402X7R104J500AT"
 			(at 199.39 81.28 0)
@@
 			(project "ARLISS_STM32_2026"
 				(path "/9719ea46-14c4-4409-9c57-49dd5454c03f/9e299f07-4887-409a-8623-587b30453872"
-					(reference "C24")
+					(reference "C27")
 					(unit 1)
 				)
