File: IMU.kicad_sch (KiCad schematic)
At the start: 1 part, among them U2 4754

Commit message: C14 y C1,C2,... modificados
Parts:
- U2: MANUFACTURER Adafruit -> (none); Manufacturer (none) -> Adafruit
Changed lines of the file:
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@@
 			)
 		)
-		(property "MANUFACTURER" "Adafruit"
+		(property "Manufacturer" "Adafruit"
 			(at 164.592 137.414 0)
 			(hide yes)
@@
 			)
 		)
+		(property "Field7" ""
+			(at 165.1 107.95 0)
+			(hide yes)
+			(show_name no)
+			(do_not_autoplace no)
+			(effects
+				(font
+					(size 1.27 1.27)
+				)
+			)
+		)

Commit message: Avance 02/08
Connections:
- net SPI1_MISO: now also U2.JP1_5 (SDA); no longer U2.JP2_5 (DI)
- net SPI1_MOSI: now also U2.JP2_5 (DI); no longer U2.JP1_5 (SDA)

Commit message: 08/08
Connections:
- net +3.3V: no longer U2.JP2_2 (P0)
- new net WAKE_BNO: U2.JP2_2 (P0)
Changed lines of the file:
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@@
 	)
 	(junction
-		(at 186.69 100.33)
-		(diameter 0)
-		(color 0 0 0 0)
-	)
-	(junction
 		(at 143.51 95.25)
 		(diameter 0)
@@
 	(wire
 		(pts
-			(xy 186.69 100.33) (xy 186.69 102.87)
+			(xy 180.34 102.87) (xy 203.2 102.87)
 		)
 		(stroke
@@
 	(wire
 		(pts
-			(xy 180.34 100.33) (xy 186.69 100.33)
-		)
-		(stroke
-			(width 0)
-			(type default)
-		)
-	)
-	(wire
-		(pts
-			(xy 180.34 102.87) (xy 186.69 102.87)
+			(xy 148.59 118.11) (xy 149.86 118.11)
 		)
 		(stroke
@@
 	(wire
 		(pts
-			(xy 148.59 118.11) (xy 149.86 118.11)
+			(xy 203.2 102.87) (xy 203.2 100.33)
 		)
 		(stroke
@@
 	(wire
 		(pts
-			(xy 191.77 100.33) (xy 186.69 100.33)
-		)
-		(stroke
-			(width 0)
-			(type default)
-		)
-	)
-	(wire
-		(pts
 			(xy 148.59 115.57) (xy 149.86 115.57)
 		)
@@
 		)
 	)
+	(global_label "WAKE_BNO"
+		(shape input)
+		(at 180.34 100.33 0)
+		(fields_autoplaced yes)
+		(effects
+			(font
+				(size 1.27 1.27)
+			)
+			(justify left)
+		)
+		(property "Intersheetrefs" "${INTERSHEET_REFS}"
+			(at 193.1828 100.33 0)
+			(hide yes)
+			(show_name no)
+			(do_not_autoplace no)
+			(effects
+				(font
+					(size 1.27 1.27)
+				)
+				(justify left)
+			)
+		)
+	)
 	(global_label "SPI1_SCLK"
 		(shape input)
@@
 	(symbol
 		(lib_id "power:+3.3V")
-		(at 191.77 100.33 0)
+		(at 203.2 100.33 0)
 		(unit 1)
 		(body_style 1)
@@
 		(fields_autoplaced yes)
 		(property "Reference" "#PWR030"
-			(at 191.77 104.14 0)
+			(at 203.2 104.14 0)
 			(hide yes)
 			(show_name no)
@@
 		)
 		(property "Value" "+3.3V"
-			(at 191.77 95.25 0)
+			(at 203.2 95.25 0)
 			(show_name no)
 			(do_not_autoplace no)
@@
 		)
 		(property "Footprint" ""
-			(at 191.77 100.33 0)
+			(at 203.2 100.33 0)
 			(hide yes)
 			(show_name no)
@@
 		)
 		(property "Datasheet" ""
-			(at 191.77 100.33 0)
+			(at 203.2 100.33 0)
 			(hide yes)
 			(show_name no)
@@
 		)
 		(property "Description" "Power symbol creates a global label with name \"+3.3V\""
-			(at 191.77 100.33 0)
+			(at 203.2 100.33 0)
 			(hide yes)
 			(show_name no)
