File: IMU.kicad_sch (KiCad schematic)
At the start: 1 part, among them U2 4754

Commit message: V3
Connections:
- net +3.3V: no longer U2.JP1_1 (VIN)
Changed lines of the file:
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@@
 		)
 	)
-	(junction
-		(at 143.51 95.25)
-		(diameter 0)
-		(color 0 0 0 0)
-	)
 	(no_connect
 		(at 180.34 95.25)
@@
 	)
 	(symbol
+		(lib_name "+3.3V_1")
 		(lib_id "power:+3.3V")
 		(at 143.51 93.98 0)
@@
 					(unit 1)
 				)
-			)
-		)
-	)
-	(symbol
-		(lib_id "power:PWR_FLAG")
-		(at 143.51 95.25 180)
-		(unit 1)
-		(body_style 1)
-		(exclude_from_sim no)
-		(in_bom yes)
-		(on_board yes)
-		(in_pos_files yes)
-		(dnp no)
-		(fields_autoplaced yes)
-		(property "Reference" "#FLG01"
-			(at 143.51 97.155 0)
-			(hide yes)
-			(show_name no)
-			(do_not_autoplace no)
-			(effects
-				(font
-					(size 1.27 1.27)
-				)
-			)
-		)
-		(property "Value" "PWR_FLAG"
-			(at 143.51 100.33 0)
-			(show_name no)
-			(do_not_autoplace no)
-			(effects
-				(font
-					(size 1.27 1.27)
-				)
-			)
-		)
-		(property "Footprint" ""
-			(at 143.51 95.25 0)
-			(hide yes)
-			(show_name no)
-			(do_not_autoplace no)
-			(effects
-				(font
-					(size 1.27 1.27)
-				)
-			)
-		)
-		(property "Datasheet" ""
-			(at 143.51 95.25 0)
-			(hide yes)
-			(show_name no)
-			(do_not_autoplace no)
-			(effects
-				(font
-					(size 1.27 1.27)
-				)
-			)
-		)
-		(property "Description" "Special symbol for telling ERC where power comes from"
-			(at 143.51 95.25 0)
-			(hide yes)
-			(show_name no)
-			(do_not_autoplace no)
-			(effects
-				(font
-					(size 1.27 1.27)
-				)
-			)
-		)
-		(pin "1"
-		)
-		(instances
-			(project "ARLISS_STM32_2026"
-				(path "/9719ea46-14c4-4409-9c57-49dd5454c03f/243e1b39-32df-463e-8f3d-bc06fe39ea80"
-					(reference "#FLG01")
-					(unit 1)
-				)

Commit message: REV_1
Connections:
- net +3.3V: now also U2.JP1_1 (VIN)
Changed lines of the file:
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@@
 	(wire
 		(pts
-			(xy 143.51 95.25) (xy 149.86 95.25)
+			(xy 137.16 95.25) (xy 149.86 95.25)
 		)
 		(stroke
@@
 	(wire
 		(pts
-			(xy 143.51 93.98) (xy 143.51 95.25)
-		)
-		(stroke
-			(width 0)
-			(type default)
-		)
-	)
-	(wire
-		(pts
 			(xy 148.59 115.57) (xy 149.86 115.57)
 		)
@@
 	)
 	(symbol
-		(lib_name "+3.3V_1")
 		(lib_id "power:+3.3V")
-		(at 143.51 93.98 0)
+		(at 137.16 95.25 0)
+		(mirror y)
 		(unit 1)
 		(body_style 1)
@@
 		(dnp no)
 		(fields_autoplaced yes)
-		(property "Reference" "#PWR028"
-			(at 143.51 97.79 0)
+		(property "Reference" "#PWR0181"
+			(at 137.16 99.06 0)
 			(hide yes)
 			(show_name no)
@@
 		)
 		(property "Value" "+3.3V"
-			(at 143.51 88.9 0)
+			(at 137.16 87.63 0)
 			(show_name no)
 			(do_not_autoplace no)
@@
 		)
 		(property "Footprint" ""
-			(at 143.51 93.98 0)
+			(at 137.16 95.25 0)
 			(hide yes)
 			(show_name no)
@@
 		)
 		(property "Datasheet" ""
-			(at 143.51 93.98 0)
+			(at 137.16 95.25 0)
 			(hide yes)
 			(show_name no)
@@
 			)
 		)
-		(property "Description" "Power symbol creates a global label with name \"+3.3V\""
-			(at 143.51 93.98 0)
-			(hide yes)
+		(property "Description" "3V3"
+			(at 137.16 90.17 0)
 			(show_name no)
 			(do_not_autoplace no)
@@
 			(project "ARLISS_STM32_2026"
 				(path "/9719ea46-14c4-4409-9c57-49dd5454c03f/243e1b39-32df-463e-8f3d-bc06fe39ea80"
-					(reference "#PWR028")
+					(reference "#PWR0181")
 					(unit 1)
 				)
