File: untitled.kicad_sch (KiCad schematic)
At the start: 0 parts

Commit message: ALIMENTACIÓN
Parts:
- added C37: 220uF, Capacitor_Tantalum_SMD:CP_EIA-7360-38_Kemet-E, symbol Device:C_Polarized_US
- added C38: 10uF, Capacitor_SMD:C_0603_1608Metric, symbol Device:C
- added C39: 330uF, Capacitor_Tantalum_SMD:CP_EIA-7343-31_Kemet-D, symbol Device:C_Polarized_US
- added C40: 4.7uF, Capacitor_SMD:C_0603_1608Metric, symbol Device:C
- added CN1, CN2: XT30PW-M, easyeda2kicad:CONN-TH_XT30PW-M, symbol easyeda2kicad:XT30PW-M
- added D4: MBRD1060, Package_TO_SOT_SMD:TO-252-2, symbol Device:D_Schottky_AKA
- added L2: 33uH, Inductor_SMD:L_APV_APH0850, symbol Device:L
- added R16: 12k, Resistor_SMD:R_0603_1608Metric, symbol Device:R
- added R17: 2.2k, Resistor_SMD:R_0603_1608Metric, symbol Device:R
- added SW1, SW2: SWITCH_BLACK, easyeda2kicad:SW-TH_XKB_SS-12M11XX, symbol CANSAT_STM32_symbols:SS-12M11G3
- added TP1, TP2, TP3: TestPoint, TestPoint:TestPoint_Pad_D1.5mm, symbol Connector:TestPoint
- added U14: XL4005, Package_TO_SOT_SMD:TO-263-5_TabPin3, symbol Regulator_Switching:XL4015
- added U15: XC6220B331MR, Package_TO_SOT_SMD:SOT-23-5, symbol Regulator_Linear:XC6220B331MR
Connections:
- new net +3V3: C40.1, TP3.1, U15.5 (VOUT)
- new net +5V: C38.1, C39.1, L2.2, R16.2, TP1.1, U15.1 (VIN), U15.3 (CE)
- new net +BATT1: CN1.2 (+), SW1.1
- new net +BATT2: CN2.2 (+), SW2.1
- new net +VIN: C37.1, SW1.2, U14.4 (VC), U14.5 (VIN)
- new net +VIN2: SW2.2
- new net FB: R16.1, R17.2, U14.2 (FB)
- new net GND: C37.2, C38.2, C39.2, C40.2, CN1.1 (-), CN2.1 (-), D4.1 (A), D4.3 (A), R17.1, SW1.3, SW2.3, TP2.1, U14.1 (GND), U15.2 (GND)
- new net SW: D4.2 (K), L2.1, U14.3 (SW)
- no-connect marks 0 -> 4

Commit message: Esquemático V1
Parts:
- removed C37: 220uF, Capacitor_Tantalum_SMD:CP_EIA-7360-38_Kemet-E, symbol Device:C_Polarized_US
- removed C39: 330uF, Capacitor_Tantalum_SMD:CP_EIA-7343-31_Kemet-D, symbol Device:C_Polarized_US
- added C10: 330uF, easyeda2kicad:CAP-TH_BD10.0-P5.00-D1.0-FD, symbol CANSAT_STM32_symbols:ECR1EPT331MLL100012
- added C8: 220uF, easyeda2kicad:CAP-TH_BD8.0-P3.50-D0.6-FD, symbol CANSAT_STM32_symbols:ECR1EBK221MLL080011
- R16: LCSC (none) -> C114659
- R17: LCSC (none) -> C114662
Connections:
- net +5V: now also C10.1
- net GND: now also C10.2
Other:
- moved on the sheet: R17, TP1, TP2, TP3

Commit message: BECERRA
Other:
- note added: "BATT_11.1V"
- note added: "BATT_7.4V"
- moved on the sheet: C10, C38, C40, C8, CN1, CN2, D4, L2, R16, R17, TP1, TP2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

Commit message: AVANCE 06
Parts:
- SW1, SW2: footprint easyeda2kicad:SW-TH_XKB_SS-12M11XX -> ARLISS-footprints:SW-TH_XKB_SS-12M11XX
Changed lines of the file:
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@@
 			)
 		)
-		(property "Footprint" "easyeda2kicad:SW-TH_XKB_SS-12M11XX"
+		(property "Footprint" "ARLISS-footprints:SW-TH_XKB_SS-12M11XX"
 			(at 74.93 74.93 0)
-			(hide yes)
 			(show_name no)
 			(do_not_autoplace no)
@@
 			)
 		)
-		(property "Footprint" "easyeda2kicad:SW-TH_XKB_SS-12M11XX"
+		(property "Footprint" "ARLISS-footprints:SW-TH_XKB_SS-12M11XX"
 			(at 74.93 43.18 0)
-			(hide yes)
-			(show_name no)
-			(do_not_autoplace no)
+			(show_name no)
+			(do_not_autoplace no)

Commit message: Parte 01 07/06
Changed lines of the file:
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@@
 	(wire
 		(pts
-			(xy 36.83 46.99) (xy 35.56 46.99)
+			(xy 36.83 46.99) (xy 33.02 46.99)
 		)
 		(stroke
@@
 	(wire
 		(pts
-			(xy 35.56 46.99) (xy 35.56 45.72)
+			(xy 33.02 46.99) (xy 33.02 44.45)
 		)
 		(stroke
@@
 	)
 	(symbol
+		(lib_name "SS-12M11G3_1")
 		(lib_id "CANSAT_STM32_symbols:SS-12M11G3")
 		(at 85.09 74.93 270)
@@
 	(symbol
 		(lib_id "power:+BATT")
-		(at 35.56 45.72 0)
+		(at 33.02 44.45 0)
 		(unit 1)
 		(body_style 1)
@@
 		(in_pos_files yes)
 		(dnp no)
-		(fields_autoplaced yes)
 		(property "Reference" "#PWR097"
-			(at 35.56 49.53 0)
+			(at 33.02 48.26 0)
 			(hide yes)
 			(show_name no)
@@
 		)
 		(property "Value" "+BATT1"
-			(at 35.56 40.64 0)
+			(at 34.29 43.18 0)
 			(show_name no)
 			(do_not_autoplace no)
@@
 					(size 1.27 1.27)
 				)
+				(justify left)
 			)
 		)
 		(property "Footprint" ""
-			(at 35.56 45.72 0)
+			(at 33.02 44.45 0)
 			(hide yes)
 			(show_name no)
@@
 		)
 		(property "Datasheet" ""
-			(at 35.56 45.72 0)
+			(at 33.02 44.45 0)
 			(hide yes)
 			(show_name no)
@@
 		)
 		(property "Description" "Power symbol creates a global label with name \"+BATT\""
-			(at 35.56 45.72 0)
+			(at 33.02 44.45 0)
 			(hide yes)
 			(show_name no)
@@
 	)
 	(symbol
+		(lib_name "XT30PW-M_1")
 		(lib_id "easyeda2kicad:XT30PW-M")
 		(at 41.91 48.26 90)

Commit message: feat: [solución de rules checker]
Parts:
- removed U14: XL4005, Package_TO_SOT_SMD:TO-263-5_TabPin3, symbol Regulator_Switching:XL4015
- added U14: XL4005E1, easyeda2kicad:TO-263-5_L10.2-W9.2-P1.70-TL, symbol CANSAT_STM32_symbols:XL4005E1
Connections:
- net +VIN: now also U14.4 (EN), U14.5 (VIN)
- net FB: now also U14.2 (FB)
- net GND: now also U14.1 (GND)
- net SW: now also U14.3 (SW), U14.6 (SW)
Other:
- moved on the sheet: C10, D4, L2, R16, R17
