File: untitled.kicad_sch (KiCad schematic)
At the start: 17 parts, among them CN1 XT30PW-M, CN2 XT30PW-M, SW1 SWITCH_BLACK, SW2 SWITCH_BLACK, U14 XL4005E1, U15 XC6220B331MR

Commit message: Cantidad de errores en la PCB: 29
Parts:
- U14: footprint easyeda2kicad:TO-263-5_L10.2-W9.2-P1.70-TL -> ARLISS-footprints:TO-263-5_L10.2-W9.2-P1.70-TL
Changed lines of the file:
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@@
 			)
 		)
-		(property "Footprint" "easyeda2kicad:TO-263-5_L10.2-W9.2-P1.70-TL"
+		(property "Footprint" "ARLISS-footprints:TO-263-5_L10.2-W9.2-P1.70-TL"
 			(at 148.59 85.09 0)
 			(hide yes)

Commit message: Cantidad de errores de la placa: 05
Parts:
- C10: footprint easyeda2kicad:CAP-TH_BD10.0-P5.00-D1.0-FD -> ARLISS-footprints:CAP-TH_BD10.0-P5.00-D1.0-FD
- C8: footprint easyeda2kicad:CAP-TH_BD8.0-P3.50-D0.6-FD -> ARLISS-footprints:CAP-TH_BD8.0-P3.50-D0.6-FD
- CN1, CN2: footprint easyeda2kicad:CONN-TH_XT30PW-M -> ARLISS-footprints:CONN-TH_XT30PW-M
Changed lines of the file:
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@@
 			)
 		)
-		(property "Footprint" "easyeda2kicad:CAP-TH_BD10.0-P5.00-D1.0-FD"
+		(property "Footprint" "ARLISS-footprints:CAP-TH_BD10.0-P5.00-D1.0-FD"
 			(at 189.23 83.82 0)
 			(hide yes)
@@
 			)
 		)
-		(property "Footprint" "easyeda2kicad:CONN-TH_XT30PW-M"
+		(property "Footprint" "ARLISS-footprints:CONN-TH_XT30PW-M"
 			(at 53.34 76.2 0)
 			(hide yes)
@@
 			)
 		)
-		(property "Footprint" "easyeda2kicad:CONN-TH_XT30PW-M"
+		(property "Footprint" "ARLISS-footprints:CONN-TH_XT30PW-M"
 			(at 53.34 48.26 0)
 			(hide yes)
@@
 			)
 		)
-		(property "Footprint" "easyeda2kicad:CAP-TH_BD8.0-P3.50-D0.6-FD"
+		(property "Footprint" "ARLISS-footprints:CAP-TH_BD8.0-P3.50-D0.6-FD"
 			(at 129.54 76.2 0)
 			(hide yes)

Commit message: PCB ordenada V1
Changed lines of the file:
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@@
 	(wire
 		(pts
-			(xy 132.08 95.25) (xy 132.08 105.41)
-		)
-		(stroke
-			(width 0)
-			(type default)
-		)
-	)
-	(wire
-		(pts
 			(xy 180.34 83.82) (xy 189.23 83.82)
 		)
@@
 	(wire
 		(pts
-			(xy 133.35 95.25) (xy 132.08 95.25)
-		)
-		(stroke
-			(width 0)
-			(type default)
-		)
-	)
-	(wire
-		(pts
 			(xy 160.02 64.77) (xy 171.45 64.77)
 		)
@@
 	(wire
 		(pts
-			(xy 133.35 93.98) (xy 133.35 95.25)
-		)
-		(stroke
-			(width 0)
-			(type default)
-		)
-	)
-	(wire
-		(pts
 			(xy 72.39 76.2) (xy 82.55 76.2)
 		)
@@
 		)
 	)
-	(symbol
-		(lib_id "power:GND")
-		(at 132.08 105.41 0)
-		(unit 1)
-		(body_style 1)
-		(exclude_from_sim no)
-		(in_bom yes)
-		(on_board yes)
-		(in_pos_files yes)
-		(dnp no)
-		(fields_autoplaced yes)
-		(property "Reference" "#PWR036"
-			(at 132.08 111.76 0)
-			(hide yes)
-			(show_name no)
-			(do_not_autoplace no)
-			(effects
-				(font
-					(size 1.27 1.27)
-				)
-			)
-		)
-		(property "Value" "GND"
-			(at 132.08 110.49 0)
-			(show_name no)
-			(do_not_autoplace no)
-			(effects
-				(font
-					(size 1.27 1.27)
-				)
-			)
-		)
-		(property "Footprint" ""
-			(at 132.08 105.41 0)
-			(hide yes)
-			(show_name no)
-			(do_not_autoplace no)
-			(effects
-				(font
-					(size 1.27 1.27)
-				)
-			)
-		)
-		(property "Datasheet" ""
-			(at 132.08 105.41 0)
-			(hide yes)
-			(show_name no)
-			(do_not_autoplace no)
-			(effects
-				(font
-					(size 1.27 1.27)
-				)
-			)
-		)
-		(property "Description" "Power symbol creates a global label with name \"GND\" , ground"
-			(at 132.08 105.41 0)
-			(hide yes)
-			(show_name no)
-			(do_not_autoplace no)
-			(effects
-				(font
-					(size 1.27 1.27)
-				)
-			)
-		)
-		(pin "1"
-		)
-		(instances
-			(project "ARLISS_STM32_2026"
-				(path "/9719ea46-14c4-4409-9c57-49dd5454c03f/8549a18f-8dc0-4c64-a4df-732ef1c8a382"
-					(reference "#PWR036")
-					(unit 1)
-				)
-			)
-		)
-	)

Commit message: Primer Ruteo de PCB
Parts:
- C38: footprint Capacitor_SMD:C_0603_1608Metric -> Capacitor_SMD:C_0603_1608Metric_Pad1.08x0.95mm_HandSolder
- R16, R17: footprint Resistor_SMD:R_0603_1608Metric -> Capacitor_SMD:C_0603_1608Metric_Pad1.08x0.95mm_HandSolder
Changed lines of the file:
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@@
 			)
 		)
-		(property "Footprint" "Capacitor_SMD:C_0603_1608Metric"
+		(property "Footprint" "Capacitor_SMD:C_0603_1608Metric_Pad1.08x0.95mm_HandSolder"
 			(at 136.8552 137.16 0)
 			(hide yes)
@@
 			)
 		)
-		(property "Footprint" "Resistor_SMD:R_0603_1608Metric"
+		(property "Footprint" "Capacitor_SMD:C_0603_1608Metric_Pad1.08x0.95mm_HandSolder"
 			(at 202.438 83.82 90)
 			(hide yes)
@@
 			)
 		)
-		(property "Footprint" "Resistor_SMD:R_0603_1608Metric"
+		(property "Footprint" "Capacitor_SMD:C_0603_1608Metric_Pad1.08x0.95mm_HandSolder"
 			(at 202.438 69.85 90)
 			(hide yes)
