File: ARLISS_STM32_2026.kicad_pcb (KiCad board)
At the start: 2 copper layers, 100 parts, among them CN1 XT30PW-M, CN2 XT30PW-M, J1 Conn_01x06, J2 Conn_01x06, J5 Screw_Terminal_01x02, Q1 IRLZ44NPBF, SW1 SWITCH_BLACK, SW2 SWITCH_BLACK, SW3 XDTD-0304-215, U1 DRV8874PWPR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

Commit message: PCB ordenada V1
Parts:
- removed U16: AP64501SP-13, ARLISS-footprints:SOIC-8_L4.9-W3.9-P1.27-LS6.0-BL-EP-1
- added C37: 100nF, ARLISS-footprints:C0402, F.Cu at (140.1, 54.7)
- added C39: 100nF, ARLISS-footprints:C0402, F.Cu at (168.6, 53.7)
- L3: value 1Kohm_100Mhz -> 1KH
- RIPROPI2, RIPROPI3: value 2.7K -> 2.4K
- moved CN1 196.6 mm to (66.0, 160.5)
- moved JP1 194.9 mm to (74.3, 41.9)
- moved CN2 194.8 mm to (82.2, 159.7)
- moved R2 187.5 mm to (62.0, 83.4)
- moved LED1 183.9 mm to (60.4, 43.5)
- moved U7 179.8 mm to (70.3, 80.1)
- moved C32 176.5 mm to (69.9, 52.7)
- moved U10 176.5 mm to (75.2, 58.0)
- moved C31 174.7 mm to (50.1, 58.2)
- moved U8 170.4 mm to (84.3, 80.0)
- moved C10 169.8 mm to (66.3, 130.9), turned to 90 degrees
- moved R1 169.4 mm to (63.0, 103.8)
- moved JP2 163.1 mm to (101.0, 60.4)
- moved C8 155.3 mm to (94.8, 132.0), turned to 90 degrees
- moved C29 151.9 mm to (61.8, 77.7)
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Connections:
- net /Motor control/IMODE1 renamed /Motor control/IMODE_1
- net /Motor control/IMODE2 renamed /Motor control/IMODE_2
- net NRST renamed /CORE_STM32F405/NRST
- C1 pad 2: nFAULT2 -> GND
- C10 pad 2: nFAULT2 -> GND
- C11 pad 1: nFAULT2 -> GND
- C13 pad 2: nFAULT2 -> GND
- C14 pad 2: nFAULT2 -> GND
- C15 pad 2: nFAULT2 -> GND
- C16 pad 2: nFAULT2 -> GND
- C17 pad 2: nFAULT2 -> GND
- C18 pad 2: nFAULT2 -> GND
- C19 pad 1: nFAULT2 -> GND
- C20 pad 1: nFAULT2 -> GND
- C21 pad 1: nFAULT2 -> GND
- C22 pad 2: nFAULT2 -> GND
- C23 pad 2: nFAULT2 -> GND
- C24 pad 2: nFAULT2 -> GND
- C25 pad 1: nFAULT2 -> GND
- C27 pad 1: nFAULT2 -> GND
- C28 pad 2: nFAULT2 -> GND
- C29 pad 1: nFAULT2 -> GND
- C3 pad 2: nFAULT2 -> GND
- C30 pad 1: nFAULT2 -> GND
- C31 pad 1: nFAULT2 -> GND
- C32 pad 2: nFAULT2 -> GND
- C34 pad 1: nFAULT2 -> GND
- C35 pad 1: nFAULT2 -> GND
- C38 pad 2: nFAULT2 -> GND
- C4 pad 2: nFAULT2 -> GND
- C40 pad 2: nFAULT2 -> GND
- C6 pad 2: nFAULT2 -> GND
- C7 pad 1: nFAULT2 -> GND
- CN1 pad 1: nFAULT2 -> GND
- CN2 pad 1: nFAULT2 -> GND
- D3 pad 2: nFAULT2 -> GND
- D4 pad 1: nFAULT2 -> GND
- D4 pad 3: nFAULT2 -> GND
- D6 pad 2: nFAULT2 -> GND
- H1 pad 1: nFAULT2 -> GND
- H1 pad 2: nFAULT2 -> GND
- J1 pad 2: nFAULT2 -> GND
- J2 pad 5: nFAULT2 -> GND
- JP1 pad 1: nFAULT2 -> GND
- JP2 pad 1: /Motor control/nFAULT1 -> nFAULT1
- LED1 pad 1: I2C2_SCL -> I2C1_SCL
- LED1 pad 3: nFAULT2 -> GND
- LED1 pad 4: I2C2_SDA -> I2C1_SDA
- Q1 pad 3: nFAULT2 -> GND
- R1 pad 2: nFAULT2 -> GND
- R17 pad 1: nFAULT2 -> GND
- R6 pad 1: nFAULT2 -> GND
- R7 pad 1: nFAULT2 -> GND
- R8 pad 1: nFAULT2 -> GND
- RIMODE1 pad 2: nFAULT2 -> GND
- RIMODE2 pad 2: nFAULT2 -> GND
- RIPROPI2 pad 2: nFAULT2 -> GND
- RIPROPI3 pad 2: nFAULT2 -> GND
- Rfault1 pad 2: nFAULT2 -> nFAULT1
- SW1 pad 3: nFAULT2 -> GND
- SW2 pad 3: nFAULT2 -> GND
- SW3 pad 2: nFAULT2 -> GND
- TP2 pad 1: nFAULT2 -> GND
- U1 pad 15: nFAULT2 -> GND
- U1 pad 17: nFAULT2 -> GND
- U1 pad 5: VREF/DAC2 -> +3V3
- U1 pad 9: nFAULT2 -> GND
- U13 pad 2: nFAULT2 -> GND
- U14 pad 1: nFAULT2 -> GND
- U15 pad 2: nFAULT2 -> GND
- U2 pad 15: nFAULT2 -> GND
- U2 pad 17: nFAULT2 -> GND
- U2 pad 4: /Motor control/nFAULT1 -> nFAULT1
- U2 pad 5: VREF/DAC1 -> +3V3
- U2 pad 9: nFAULT2 -> GND
- U3 pad JP1_3: nFAULT2 -> GND
- U4 pad 10: VREF/DAC2 -> nFAULT2
- U4 pad 11: VREF/DAC1 -> nFAULT1
- U4 pad 12: nFAULT2 -> GND
- U4 pad 18: nFAULT2 -> GND
- U4 pad 2: unconnected-(U4A-PC13-Pad2) -> IMU INT
- U4 pad 24: unconnected-(U4A-PC4-Pad24) -> DPS_INT
- U4 pad 29: I2C2_SCL -> unconnected-(U4A-PB10-Pad29)
- U4 pad 30: I2C2_SDA -> unconnected-(U4A-PB11-Pad30)
- U4 pad 53: PIN_MOSFET -> unconnected-(U4A-PC12-Pad53)
- U4 pad 57: DPS_INT -> unconnected-(U4A-PB5-Pad57)
- U4 pad 61: IMU INT -> PIN_MOSFET
- U4 pad 63: nFAULT2 -> GND
- U5 pad 1: nFAULT2 -> GND
- U5 pad 7: nFAULT2 -> GND
- U6 pad 12: nFAULT2 -> GND
- U6 pad 13: nFAULT2 -> GND
- U6 pad 16: nFAULT2 -> GND
- U7 pad 1: nFAULT2 -> GND
- U7 pad 2: nFAULT2 -> GND
- U7 pad 4: I2C2_SDA -> I2C1_SDA
- U7 pad 5: I2C2_SCL -> I2C1_SCL
- U7 pad 7: nFAULT2 -> GND
- U8 pad 1: nFAULT2 -> GND
- U8 pad 4: I2C2_SDA -> I2C1_SDA
- U8 pad 5: I2C2_SCL -> I2C1_SCL
- U8 pad 7: nFAULT2 -> GND
- U9 pad 2: nFAULT2 -> GND
- X2 pad 2: nFAULT2 -> GND
Other:
- copper layers 2 -> 4

Commit message: DPS ORDENADO
Parts:
- L3: value 1KH -> 1Kohm_100Mhz
- moved C8 75.9 mm to (40.7, 185.2), turned to -90 degrees
- moved L2 63.4 mm to (31.2, 166.0)
- moved R17 63.3 mm to (40.7, 167.7)
- moved R16 56.1 mm to (40.7, 162.5)
- moved D4 53.5 mm to (31.0, 181.9)
- moved C1 51.1 mm to (221.7, 34.8)
- moved C2 51.1 mm to (220.6, 38.4)
- moved C3 51.1 mm to (209.8, 23.3)
- moved C33 51.1 mm to (234.7, 37.4)
- moved C34 51.1 mm to (234.7, 39.5)
- moved C39 51.1 mm to (217.3, 38.3)
- moved D3 51.1 mm to (209.3, 34.0)
- moved J1 51.1 mm to (222.2, 24.5)
- moved JP3 51.1 mm to (210.1, 48.2)
- moved RIMODE2 51.1 mm to (234.6, 46.2)
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Connections:
- C8 pad 1: unconnected-(C8-Pad1) -> +VIN
- C8 pad 2: unconnected-(C8-Pad2) -> GND

Commit message: Driver Ordenado
Parts:
- moved C37 21.9 mm to (155.0, 38.6)
- moved C4 21.9 mm to (129.3, 24.8)
- moved C5 21.9 mm to (146.8, 32.3)
- moved C6 21.9 mm to (127.9, 48.6)
- moved J2 21.9 mm to (139.9, 21.2)
- moved JP2 21.9 mm to (115.9, 44.3)
- moved D6 21.9 mm to (128.9, 36.2)
- moved RIMODE1 21.9 mm to (156.0, 49.5)
- moved RIPROPI3 21.9 mm to (150.6, 48.5)
- moved U2 21.9 mm to (147.5, 38.7)
- moved C35 21.9 mm to (137.9, 39.4)
- moved C36 21.9 mm to (137.9, 41.5)
- moved RLED1 21.9 mm to (117.5, 31.7)
- moved Rfault1 21.9 mm to (138.9, 31.9)
- moved U11 21.9 mm to (116.4, 36.7)
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Connections:
- C8 pad 1: +VIN -> unconnected-(C8-Pad1)
- C8 pad 2: GND -> unconnected-(C8-Pad2)
Routing:
- net nFAULT2: track 0.00 -> 6.98 mm
- net +VIN2: track 0.00 -> 6.32 mm
- net /Motor control/M2+: track 0.00 -> 5.55 mm
- net /Motor control/IMODE_2: track 0.00 -> 3.96 mm
- net +3V3: track 0.00 -> 3.66 mm
- net ADC2: track 0.00 -> 3.56 mm
- net Net-(U1-CPL): track 0.00 -> 2.60 mm
- net Net-(JP3-B): track 0.00 -> 2.57 mm
- net /Motor control/VCP2: track 0.00 -> 2.47 mm
- net Net-(U1-CPH): track 0.00 -> 2.40 mm
