File: ARLISS_STM32_2026.kicad_pcb (KiCad board)
At the start: 4 copper layers, 123 parts, among them CN1 XT30PW-M, CN2 XT30PW-M, CN4 0430450400, J1 Conn_01x06, J2 Conn_01x06, J3 Screw_Terminal_01x02, P1 PZ254R-12-8P, Q1 IRLZ44NPBF, Q2 AOD4185_C400894, Q3 AOD4185_C400894, SW1 EVQPLMA15, SW2 EVQPLMA15, SW3 SWITCH_BLACK, SW4 SWITCH_BLACK, U1 STM32F405RGT6, U10 INA226AIDGSR, U11 INA226AIDGSR, U12 ADXL375BCCZ, U2 4754, U3 DRV8874PWPR, U4 DRV8874PWPR, U5 BMP581, U6 VEML7700-TR, U7 TPS62901RPJR, X1 32.768kHz 7pF SMD, X2 8Mhz 10pF

Commit message: Cambios finales antes de main
Parts:
- removed D2: SMBJ18A_C151256, ARLISS-footprints:SMB_L4.3-W3.6-LS5.3-RD
- added D5: SMBJ18CA_C83327, ARLISS-footprints:SMB_L4.6-W3.6-LS5.3-BI, F.Cu at (72.1, 69.3)
- added D6: SMBJ18CA_C83327, ARLISS-footprints:SMB_L4.6-W3.6-LS5.3-BI, F.Cu at (167.7, 90.0)
- added JP1: SolderJumper_2_Open, Jumper:SolderJumper-2_P1.3mm_Open_TrianglePad1.0x1.5mm, F.Cu at (82.2, 101.0)
- added JP2: SolderJumper_2_Open, Jumper:SolderJumper-2_P1.3mm_Open_TrianglePad1.0x1.5mm, F.Cu at (156.4, 97.5)
- added JP3: SolderJumper_2_Open, Jumper:SolderJumper-2_P1.3mm_Open_TrianglePad1.0x1.5mm, F.Cu at (153.2, 104.0)
- added JP4: SolderJumper_2_Open, Jumper:SolderJumper-2_P1.3mm_Open_TrianglePad1.0x1.5mm, F.Cu at (82.3, 96.9)
- added LED6: ~, Diode_SMD:D_0603_1608Metric_Pad1.05x0.95mm_HandSolder, F.Cu at (160.9, 97.2)
- added LED7: ~, Diode_SMD:D_0603_1608Metric_Pad1.05x0.95mm_HandSolder, F.Cu at (158.3, 100.2)
- added LED8: ~, Diode_SMD:D_0603_1608Metric_Pad1.05x0.95mm_HandSolder, F.Cu at (77.6, 97.0)
- added R31: 2.4K, Resistor_SMD:R_0603_1608Metric_Pad0.98x0.95mm_HandSolder, F.Cu at (92.7, 57.5)
- added R32: 2.4K, Resistor_SMD:R_0603_1608Metric_Pad0.98x0.95mm_HandSolder, F.Cu at (72.0, 97.1)
- added R33: 4.7K, Resistor_SMD:R_0603_1608Metric_Pad0.98x0.95mm_HandSolder, F.Cu at (163.9, 101.3)
- added TP5: TestPoint, TestPoint:TestPoint_Pad_D1.5mm, F.Cu at (169.7, 101.2)
- C39, C40, C46, C47, D3, D4, F1, F2, Q2, Q3, R11, R20, R21, R22, R23, R24, R25, R26, R27, R28, U10, U11: moved to B.Cu
- D1: value SMBJ18A_C151256 -> SMBJ10A_C151250; footprint ARLISS-footprints:SMB_L4.3-W3.6-LS5.3-RD -> ARLISS-footprints:SMB_L4.6-W3.6-LS5.3-RD; moved to B.Cu
- Q1: footprint ARLISS-footprints:TO-220-3_L10.0-W4.5-P2.54-T -> Package_TO_SOT_THT:TO-220-3_Horizontal_TabDown
- R10, R4, R9: value 1K -> 2.4K
- R17: value 1k -> 2.4K
- moved TP1 119.3 mm to (169.6, 97.1)
- moved Q2 108.7 mm to (141.1, 111.5), turned to -90 degrees
- moved R29 105.8 mm to (133.5, 100.9)
- moved F1 96.0 mm to (134.7, 110.5), turned to 90 degrees
- moved R16 92.7 mm to (165.8, 97.2), turned to 0 degrees
- moved C40 81.6 mm to (154.0, 114.5), turned to -90 degrees
- moved U11 81.6 mm to (158.3, 114.4), turned to 180 degrees
- moved R21 81.4 mm to (158.2, 119.2), turned to 0 degrees
- moved D1 76.8 mm to (72.4, 110.1), turned to 180 degrees
- moved R27 73.9 mm to (147.5, 110.5), turned to 90 degrees
- moved R30 71.4 mm to (82.5, 110.1), turned to 180 degrees
- moved D3 68.4 mm to (141.4, 118.5)
- moved TP4 67.2 mm to (61.7, 100.6)
- moved Q3 63.7 mm to (78.6, 121.3), turned to -90 degrees
- moved TP2 61.3 mm to (61.5, 97.1)
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Connections:
- C15 pad 1: +3V3 -> +3.3V
- C16 pad 1: +3V3 -> +3.3V
- C21 pad 1: +VIN2 -> +11.1V
- C22 pad 1: +VIN2 -> +11.1V
- C23 pad 2: +VIN2 -> +11.1V
- C24 pad 2: +VIN2 -> +11.1V
- C25 pad 2: +VIN2 -> +11.1V
- C26 pad 2: +VIN2 -> +11.1V
- C27 pad 2: +3V3 -> +3.3V
- C39 pad 2: +3V3 -> +3.3V
- C40 pad 2: +3V3 -> +3.3V
- C42 pad 1: +3V3 -> +3.3V
- C45 pad 1: +3V3 -> +3.3V
- C46 pad 1: Net-(C46-Pad1) -> +VINP
- C47 pad 1: VIN2+ -> +VIN2P
- C47 pad 2: VINS2+ -> +11.1V
- D1 pad 1: +VIN2 -> +VINP
- J1 pad 5: +3V3 -> +3.3V
- J2 pad 5: +3V3 -> +3.3V
- J3 pad 1: +VIN2 -> +11.1V
- LED4 pad 1: GND -> Net-(JP1-A)
- R10 pad 1: Net-(LED3-+) -> +3.3V
- R10 pad 2: +3V3 -> Net-(LED3-+)
- R11 pad 1: Net-(C46-Pad1) -> +VINP
- R12 pad 1: +3V3 -> +3.3V
- R15 pad 2: +3V3 -> +3.3V
- R16 pad 1: Net-(LED4-+) -> Net-(LED6-+)
- R16 pad 2: +3.3V -> +11.1V
- R17 pad 1: Net-(LED5-+) -> PIN_MOSFET
- R17 pad 2: PIN_MOSFET -> Net-(LED5-+)
- R20 pad 2: +3V3 -> +3.3V
- R21 pad 2: +3V3 -> +3.3V
- R22 pad 1: VIN2+ -> +VIN2P
- R22 pad 2: VINS2+ -> +11.1V
- R23 pad 1: Net-(C46-Pad1) -> +VINP
- R25 pad 1: VIN2+ -> +VIN2P
- R26 pad 1: VINS2+ -> +11.1V
- R4 pad 1: Net-(LED1-+) -> +3.3V
- R4 pad 2: +3.3V -> Net-(LED4-+)
- R9 pad 1: Net-(LED2-+) -> +3.3V
- R9 pad 2: +3V3 -> Net-(LED2-+)
- SW1 pad 1: /CORE_STM32F405/NRST -> GND
- SW1 pad 3: GND -> /CORE_STM32F405/NRST
- SW2 pad 1: Net-(R2-Pad1) -> GND
- SW2 pad 3: GND -> Net-(R2-Pad1)
- TP1 pad 1: +VIN2 -> +11.1V
- TP4 pad 1: +3V3 -> +3.3V
- U1 pad 57: unconnected-(U1A-PB5-Pad57) -> WAKE_BNO
- U10 pad 6: +3V3 -> +3.3V
- U11 pad 2: +3V3 -> +3.3V
- U11 pad 6: +3V3 -> +3.3V
- U11 pad 8: VIN2+ -> +11.1V
- U12 pad 1: +3V3 -> +3.3V
- U2 pad JP2_2: +3.3V -> WAKE_BNO
- U3 pad 11: +VINS2 -> +11.1V
- U3 pad 16: +3V3 -> +3.3V
- U3 pad 5: +3V3 -> +3.3V
- U4 pad 11: +VINS2 -> +11.1V
- U4 pad 16: +3V3 -> +3.3V
- U4 pad 5: +3V3 -> +3.3V

Commit message: PCB_2.0
Parts:
- removed JP2: SolderJumper_2_Open, Jumper:SolderJumper-2_P1.3mm_Open_TrianglePad1.0x1.5mm
- removed LED6: ~, Diode_SMD:D_0603_1608Metric_Pad1.05x0.95mm_HandSolder
- removed R32, RIPROPI1, RIPROPI2: 2.4K, Resistor_SMD:R_0603_1608Metric_Pad0.98x0.95mm_HandSolder
- removed R33: 4.7K, Resistor_SMD:R_0603_1608Metric_Pad0.98x0.95mm_HandSolder
- removed RIMODE1, RIMODE2: 20K, Resistor_SMD:R_0603_1608Metric_Pad0.98x0.95mm_HandSolder
- added R34: 4.7K, Resistor_SMD:R_0603_1608Metric_Pad0.98x0.95mm_HandSolder, F.Cu at (76.8, 100.9)
- added RIM1: 20K, Resistor_SMD:R_0603_1608Metric_Pad0.98x0.95mm_HandSolder, F.Cu at (159.4, 85.3)
- added RIM2: 20K, Resistor_SMD:R_0603_1608Metric_Pad0.98x0.95mm_HandSolder, F.Cu at (74.1, 71.7)
- added RIPR1: 2.4K, Resistor_SMD:R_0603_1608Metric_Pad0.98x0.95mm_HandSolder, F.Cu at (70.6, 74.3)
- added RIPR2: 2.4K, Resistor_SMD:R_0603_1608Metric_Pad0.98x0.95mm_HandSolder, F.Cu at (151.1, 76.6)
- added TP6: TestPoint, TestPoint:TestPoint_Pad_D1.5mm, F.Cu at (136.0, 125.4)
- R16: value 4.7K -> 10K
- moved D5 94.8 mm to (164.9, 88.9)
- moved D6 83.9 mm to (83.9, 92.9), turned to -90 degrees
- moved SW1 64.2 mm to (106.1, 115.6)
- moved U5 47.2 mm to (91.1, 86.1)
- moved R2 43.6 mm to (131.4, 63.4), turned to -90 degrees
- moved C28 43.4 mm to (136.2, 63.4), turned to -90 degrees
- moved TP1 41.2 mm to (136.0, 120.9)
- moved R31 38.9 mm to (122.6, 82.4)
- moved H1 38.0 mm to (82.0, 141.5)
- moved C30 37.3 mm to (88.3, 77.8), turned to 90 degrees
- moved TP5 37.2 mm to (136.0, 117.0)
- moved C44 34.1 mm to (87.5, 88.2)
- moved C43 33.3 mm to (87.5, 84.7)
- moved J3 30.6 mm to (158.9, 99.8)
- moved R26 29.3 mm to (138.4, 130.5), turned to 180 degrees
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Connections:
- JP1 pad 1: Net-(JP1-A) -> +3.3V
- JP1 pad 2: GND -> Net-(JP1-B)
- JP3 pad 1: Net-(JP3-A) -> +VIN2
- JP3 pad 2: GND -> Net-(JP3-B)
- JP4 pad 1: Net-(JP4-A) -> +VIN
- JP4 pad 2: GND -> Net-(JP4-B)
- LED4 pad 1: Net-(JP1-A) -> GND
- LED7 pad 1: Net-(JP3-A) -> GND
- LED8 pad 1: Net-(JP4-A) -> GND
- R16 pad 1: Net-(LED6-+) -> Net-(LED7-+)
- R16 pad 2: +11.1V -> Net-(JP3-B)
- R4 pad 1: +3.3V -> Net-(JP1-B)

Commit message: jhamir
Parts:
- removed H6: MountingHole, MountingHole:MountingHole_3.2mm_M3_ISO14580_Pad
- moved LED5 61.6 mm to (138.9, 119.9)
- moved CN4 58.6 mm to (108.6, 121.9), turned to 0 degrees
- moved H3 53.9 mm to (125.5, 97.5)
- moved R2 51.1 mm to (84.2, 83.1)
- moved R3 51.1 mm to (86.7, 83.1)
- moved SW2 51.1 mm to (86.7, 77.5)
- moved C28 51.1 mm to (89.0, 83.1)
- moved H4 47.8 mm to (161.9, 73.4)
- moved TP6 46.4 mm to (162.6, 87.4)
- moved TP1 45.9 mm to (162.5, 83.4)
- moved TP5 45.9 mm to (162.5, 79.5)
- moved C21 43.4 mm to (141.3, 104.2), turned to 180 degrees
- moved D5 37.3 mm to (131.3, 105.2), turned to -90 degrees
- moved C23 36.6 mm to (141.0, 99.1)
- moved R9 36.1 mm to (144.6, 110.5), turned to 180 degrees
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Routing:
- net +VIN: track 0.00 -> 7.92 mm
- added copper zone on In2.Cu, net (none)
- added copper zone on In2.Cu, net +BATT1
- added copper zone on In2.Cu, net +VIN

Commit message: ordenando
Parts:
- removed C33: 4.7nF, Capacitor_SMD:C_0603_1608Metric_Pad1.08x0.95mm_HandSolder
- removed D3, D4: D_Zener, Diode_SMD:D_SOD-123
- removed D5, D6: SMBJ18CA_C83327, ARLISS-footprints:SMB_L4.6-W3.6-LS5.3-BI
- removed JP1, JP3, JP4: SolderJumper_2_Open, Jumper:SolderJumper-2_P1.3mm_Open_TrianglePad1.0x1.5mm
- removed L2: 1uH, ARLISS-footprints:IND-SMD_L4.0-W4.0_XAL4030-332MEC
- removed LED8: ~, Diode_SMD:D_0603_1608Metric_Pad1.05x0.95mm_HandSolder
- removed R13: 76.8k, Resistor_SMD:R_0603_1608Metric_Pad0.98x0.95mm_HandSolder
- removed R14: 249k, Resistor_SMD:R_0603_1608Metric_Pad0.98x0.95mm_HandSolder
- removed R27, R28: 100k, Resistor_SMD:R_0603_1608Metric_Pad0.98x0.95mm_HandSolder
- removed R29, R30: TLRZ2ATTD, ARLISS-footprints:R0805
- removed R34: 4.7K, Resistor_SMD:R_0603_1608Metric_Pad0.98x0.95mm_HandSolder
- removed SW3, SW4: SWITCH_BLACK, ARLISS-footprints:SW-TH_XKB_SS-12M11XX
- removed TP1, TP2, TP3, TP4, TP5, TP6: TestPoint, TestPoint:TestPoint_Pad_D1.5mm
- removed U7: TPS62901RPJR, ARLISS-footprints:VQFN-HR-9_L2.0-W1.5-P0.50-BL_TI_RPJ
- added D2: D_Zener, Diode_SMD:D_SOD-123, F.Cu at (121.8, 131.6)
- added R32: 100k, Resistor_SMD:R_0603_1608Metric_Pad0.98x0.95mm_HandSolder, F.Cu at (116.2, 126.9)
- added R33: 100k, Resistor_SMD:R_0603_1608Metric_Pad0.98x0.95mm_HandSolder, F.Cu at (71.0, 125.3)
- added TP10: TestPoint, TestPoint:TestPoint_Pad_D1.5mm, F.Cu at (121.7, 115.2)
- added TP11: TestPoint, TestPoint:TestPoint_Pad_D1.5mm, F.Cu at (61.7, 109.9)
- added TP12: TestPoint, TestPoint:TestPoint_Pad_D1.5mm, F.Cu at (61.7, 113.5)
- added TP9: TestPoint, TestPoint:TestPoint_Pad_D1.5mm, F.Cu at (121.7, 111.7)
- C31: value 22uF -> 10uF
- D1: value SMBJ10A_C151250 -> D_Zener; footprint ARLISS-footprints:SMB_L4.6-W3.6-LS5.3-RD -> Diode_SMD:D_SOD-123; moved to F.Cu
- F1, F2, Q2, Q3: moved to F.Cu
- R10, R17, R31, R4, R9, RIPR1, RIPR2: value 2.4K -> 2.2K
- moved Q2 73.3 mm to (75.8, 122.8)
- moved R12 59.8 mm to (110.2, 148.3)
- moved C29 59.8 mm to (112.1, 152.6)
- moved C30 59.8 mm to (108.7, 152.6)
- moved U6 59.8 mm to (115.2, 151.1)
- moved F1 53.5 mm to (88.7, 116.2), turned to 0 degrees
- moved CN4 52.0 mm to (123.9, 72.2)
- moved H3 48.9 mm to (174.4, 97.5)
- moved Q3 44.4 mm to (121.6, 124.5)
- moved C28 40.1 mm to (126.0, 98.8)
- moved R2 40.1 mm to (121.2, 98.8)
- moved R3 40.1 mm to (123.6, 98.8)
- moved SW2 40.1 mm to (123.6, 93.2)
- moved LED7 37.9 mm to (130.8, 111.8)
- moved R16 37.7 mm to (125.9, 111.8)
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Connections:
- C31 pad 2: +3.3V -> +11.1V
- C32 pad 2: Net-(U7-EN) -> +11.1V
- CN1 pad 2: +BATT1 -> +BATT2
- CN2 pad 2: +BATT2 -> +BATT1
- D1 pad 1: +VINP -> +VIN2P
- D1 pad 2: GND -> Net-(D1-A)
- F1 pad 2: +VIN2 -> +BATT2
- F2 pad 2: +VIN -> +BATT1
- Q2 pad 1: Net-(D3-A) -> Net-(D1-A)
- R16 pad 2: Net-(JP3-B) -> +11.1V
- R4 pad 1: Net-(JP1-B) -> +3.3V
Routing:
- net +VIN: track 7.92 -> 0.00 mm
- removed copper zone on In2.Cu, net +VIN

Commit message: pcb order
Parts:
- removed H3: MountingHole, MountingHole:MountingHole_3.2mm_M3_ISO14580_Pad
- D1, D2, Q2, Q3, R32, R33: moved to B.Cu
- moved U6 57.5 mm to (89.7, 99.6), turned to 180 degrees
- moved C29 54.1 mm to (91.2, 102.7), turned to 180 degrees
- moved C32 53.7 mm to (131.4, 106.2), turned to 180 degrees
- moved C30 49.7 mm to (91.2, 106.1), turned to 180 degrees
- moved R12 49.6 mm to (86.9, 104.6), turned to 90 degrees
- moved Q1 20.9 mm to (152.7, 112.8), turned to 180 degrees
- moved R2 19.6 mm to (122.5, 79.2)
- moved R3 19.6 mm to (125.0, 79.2)
- moved SW2 19.6 mm to (125.0, 73.5)
- moved C28 19.6 mm to (127.3, 79.2)
- moved R4 18.4 mm to (74.7, 126.3)
- moved LED4 18.4 mm to (79.2, 126.3)
- moved TP11 18.4 mm to (70.0, 126.3)
- moved TP12 18.4 mm to (70.0, 129.8)
- moved C43 17.2 mm to (86.7, 89.7)
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
Commit message: ARREGLOS
Parts:
- C15, C16, C17, C18, C19, C20, C23, C24, C25, C26, C31, C32, RIM1, RIM2, RIPR1, RIPR2, U3, U4: moved to B.Cu
- moved C39 75.7 mm to (145.4, 119.5), turned to 180 degrees
- moved R20 69.8 mm to (145.4, 115.2), turned to 0 degrees
- moved R24 68.4 mm to (141.1, 122.8), turned to 90 degrees
- moved SW2 66.9 mm to (86.2, 128.1), turned to -90 degrees
- moved U10 66.0 mm to (141.6, 117.3), turned to 0 degrees
- moved C28 61.4 mm to (83.8, 122.5), turned to 90 degrees
- moved R21 60.6 mm to (72.3, 111.4), turned to -90 degrees
- moved R11 60.0 mm to (138.9, 126.8), turned to 0 degrees
- moved R3 58.1 mm to (86.2, 122.5), turned to -90 degrees
- moved C46 57.4 mm to (136.6, 122.8), turned to -90 degrees
- moved J1 56.9 mm to (116.0, 72.5), turned to 0 degrees
- moved CN4 56.3 mm to (74.2, 121.2), turned to 0 degrees
- moved U11 55.5 mm to (77.1, 111.8), turned to 90 degrees
- moved R23 55.5 mm to (136.7, 118.6)
- moved R2 55.0 mm to (88.7, 122.5), turned to 90 degrees
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
Commit message: 3D MODEL
Parts:
- removed J3: Screw_Terminal_01x02, TerminalBlock_RND:TerminalBlock_RND_205-00232_1x02_P5.08mm_Horizontal
- removed TP10, TP11, TP12, TP9: TestPoint, TestPoint:TestPoint_Pad_D1.5mm
- added CN3: DB127V-5.08-2P-GN-S, ARLISS-footprints:CONN-TH_2P-P5.08, F.Cu at (137.9, 102.2)
- added TP1: TestPoint, TestPoint:TestPoint_Pad_D1.5mm, F.Cu at (75.5, 114.7)
- added TP2: TestPoint, TestPoint:TestPoint_Pad_D1.5mm, F.Cu at (126.6, 115.2)
- added TP3: TestPoint, TestPoint:TestPoint_Pad_D1.5mm, F.Cu at (137.5, 115.2)
- added TP4: TestPoint, TestPoint:TestPoint_Pad_D1.5mm, F.Cu at (86.8, 114.8)
- moved R18 17.5 mm to (137.3, 92.7), turned to 180 degrees
- moved R19 13.6 mm to (133.4, 92.7)
- moved LED7 12.6 mm to (133.9, 115.2)
- moved R16 11.7 mm to (130.0, 115.2)
- moved C45 7.72 mm to (72.5, 71.0), turned to 0 degrees
- moved R20 7.06 mm to (138.6, 113.3), turned to 180 degrees
- moved LED4 6.45 mm to (83.1, 114.8)
- moved R4 6.45 mm to (79.2, 114.8)
- moved F2 5.89 mm to (118.8, 114.5)
- moved C39 5.83 mm to (140.6, 122.6), turned to 90 degrees
- moved C21 5.60 mm to (126.5, 83.0)
- moved C27 5.12 mm to (71.0, 75.5), turned to 90 degrees
- moved C15 5.05 mm to (111.1, 82.1)
- moved C18 5.05 mm to (111.1, 80.4)
- moved C20 5.05 mm to (123.2, 84.0)
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
Commit message: Primer_plano
Parts:
- moved R11 57.0 mm to (82.1, 111.2), turned to 90 degrees
- moved R22 52.6 mm to (134.8, 118.9), turned to 90 degrees
- moved F2 21.9 mm to (97.0, 114.6), turned to 0 degrees
- moved F1 21.8 mm to (118.8, 114.3), turned to 180 degrees
- moved LED7 8.65 mm to (136.2, 123.6)
- moved R16 8.65 mm to (132.3, 123.6)
- moved TP2 8.65 mm to (128.8, 123.6)
- moved TP3 8.65 mm to (139.7, 123.6)
- moved C46 6.41 mm to (138.2, 117.5), turned to 90 degrees
- moved R23 5.94 mm to (139.2, 122.4), turned to 90 degrees
- moved R26 5.00 mm to (78.7, 109.7)
- moved R25 4.18 mm to (78.6, 112.8)
- moved R24 2.48 mm to (141.1, 122.4)
- moved C39 2.44 mm to (143.0, 122.4)
- moved U10 2.44 mm to (142.0, 117.2)
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Connections:
- C46 pad 2: Net-(C46-Pad2) -> +11.1V
- C47 pad 2: +11.1V -> +3.3V
- F1 pad 1: Net-(Q2-D) -> Net-(Q3-D)
- F1 pad 2: +BATT2 -> +BATT1
- F2 pad 1: Net-(Q3-D) -> Net-(Q2-D)
- F2 pad 2: +BATT1 -> +BATT2
- R11 pad 1: +VINP -> +VIN2P
- R11 pad 2: Net-(C46-Pad2) -> +3.3V
- R22 pad 1: +VIN2P -> +VINP
- R24 pad 1: Net-(C46-Pad2) -> +11.1V
- R26 pad 1: +11.1V -> +3.3V
- U10 pad 8: Net-(U10-VBUS) -> +11.1V
- U11 pad 8: +11.1V -> +3.3V
Routing:
- net +VIN2P: track 0.00 -> 15.7 mm
- net Net-(Q2-D): track 0.00 -> 13.4 mm, vias 0 -> 4
- net +BATT2: track 0.00 -> 5.72 mm, vias 0 -> 2
- net Net-(D1-A): track 0.00 -> 4.41 mm
- net Net-(U11-VIN-): track 0.00 -> 4.39 mm
- net Net-(U11-VIN+): track 0.00 -> 2.39 mm
- net ALERT2_INA226: track 0.00 -> 2.23 mm
- net +BATT1: vias 0 -> 1
- added copper zone on In2.Cu, net +3.3V
- added copper zone on In2.Cu, net +BATT2
- added copper zone on In2.Cu, net Net-(Q2-D)
- removed copper zone on In2.Cu, net (none)
- removed copper zone on In2.Cu, net +BATT1
Other:
- board text added: "+"
- board text added: "-"
- board text added: "TOMEK TEAM"
- board text added: "x"
- board text added: "y"
- board text added: "z"
