File: ARLISS_STM32_2026.kicad_pcb (KiCad board)
At the start: 4 copper layers, 112 parts, among them CN1 XT30PW-M, CN2 XT30PW-M, CN3 DB127V-5.08-2P-GN-S, CN4 0430450400, J1 Conn_01x06, J2 Conn_01x06, P1 PZ254R-12-8P, Q1 IRLZ44NPBF, Q2 AOD4185_C400894, Q3 AOD4185_C400894, SW1 EVQPLMA15, SW2 EVQPLMA15, U1 STM32F405RGT6, U10 INA226AIDGSR, U11 INA226AIDGSR, U12 ADXL375BCCZ, U2 4754, U3 DRV8874PWPR, U4 DRV8874PWPR, U5 BMP581, U6 VEML7700-TR, X1 32.768kHz 7pF SMD, X2 8Mhz 10pF

Commit message: pcb_v2
Parts:
- moved LED7 12.2 mm to (136.2, 111.4)
- moved R16 12.2 mm to (132.3, 111.4)
- moved TP2 12.2 mm to (128.8, 111.4)
- moved TP3 12.2 mm to (139.7, 111.4)
- moved R32 8.00 mm to (127.4, 116.3), turned to 180 degrees
- moved F2 0.76 mm to (96.2, 114.6)
- moved F1 0.50 mm to (119.2, 114.5)
Routing:
- net Net-(Q2-D): track 13.4 -> 0.01 mm, vias 4 -> 0
- net Net-(D2-A): track 0.00 -> 5.95 mm
- net +BATT2: track 5.72 -> 0.00 mm, vias 2 -> 0
- net Net-(U10-VIN+): track 0.00 -> 3.15 mm
- net Net-(U10-VIN-): track 0.00 -> 2.35 mm
- net +3.3V: track 0.00 -> 2.26 mm
- net ALERT1_INA226: track 0.00 -> 2.09 mm
- net Net-(Q3-D): vias 0 -> 3
- net +BATT1: vias 1 -> 0
- added copper zone on In2.Cu, net +11.1V
- added copper zone on F.Cu, net +BATT1
- added copper zone on In2.Cu, net +BATT1
- added copper zone on F.Cu, net +BATT2
- added copper zone on B.Cu, net +VINP
- added copper zone on B.Cu, net Net-(Q2-D)
- added copper zone on F.Cu, net Net-(Q2-D)
- added copper zone on B.Cu, net Net-(Q3-D)
- added copper zone on F.Cu, net Net-(Q3-D)
- added copper zone on In2.Cu, net Net-(Q3-D)

Commit message: V3
Parts:
- added C2: 100nF, Capacitor_SMD:C_0603_1608Metric_Pad1.08x0.95mm_HandSolder, B.Cu at (68.4, 96.1)
- added C33: 10uF, Capacitor_SMD:C_0805_2012Metric_Pad1.18x1.45mm_HandSolder, B.Cu at (75.0, 100.7)
- added C34: 22uF, Capacitor_SMD:C_0805_2012Metric_Pad1.18x1.45mm_HandSolder, B.Cu at (65.5, 102.8)
- added C35: 22uF, Capacitor_SMD:C_0805_2012Metric_Pad1.18x1.45mm_HandSolder, B.Cu at (75.0, 98.3)
- added L2: 3.3uH, ARLISS-footprints:IND-SMD_L4.1-W4.1_FTC404020S, B.Cu at (65.8, 99.3)
- added U7: AP63203QWU-7, ARLISS-footprints:TSOT-26_L2.9-W1.6-P0.95-LS2.8-BL, B.Cu at (70.5, 99.3)
- moved C40 0.40 mm to (74.5, 109.0)
Connections:
- C47 pad 2: +3.3V -> VINS+
- CN4 pad 1: GND -> /CORE_STM32F405/RADXA_PIN
- R11 pad 2: +3.3V -> VINS+
- R26 pad 1: +3.3V -> VINS+
- U11 pad 8: +3.3V -> VINS+
- U2 pad JP1_1: +3.3V -> Net-(U2-VIN)
Routing:
- net +VIN2P: track 15.7 -> 0.12 mm
- net Net-(U11-VIN-): track 4.39 -> 0.00 mm
- net Net-(D1-A): track 4.41 -> 7.42 mm
- net Net-(Q2-D): vias 0 -> 3
- added copper zone on B.Cu, net +VIN2P
- removed copper zone on In2.Cu, net +3.3V

Commit message: REV_1
Parts:
- moved R11 8.35 mm to (73.7, 111.2)
- moved C40 8.35 mm to (66.1, 109.0)
- moved C47 8.35 mm to (76.3, 111.3)
- moved R25 8.35 mm to (70.3, 112.8)
- moved R26 8.35 mm to (70.3, 109.7)
- moved U11 8.35 mm to (64.9, 111.8)
- moved C34 7.18 mm to (63.4, 95.9), turned to 0 degrees
- moved R21 5.65 mm to (63.6, 114.8), turned to 0 degrees
- moved C33 4.62 mm to (70.7, 102.3), turned to 0 degrees
- moved C20 3.17 mm to (120.7, 85.8)
- moved C19 2.75 mm to (97.3, 85.2)
- moved C39 2.68 mm to (144.4, 120.2)
- moved U6 2.50 mm to (66.0, 103.4)
- moved C30 2.44 mm to (66.4, 101.0)
- moved R19 2.35 mm to (131.6, 94.2), turned to 90 degrees
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Connections:
- C33 pad 2: Net-(U7-EN) -> +VDC
- C47 pad 2: VINS+ -> +VDC
- R11 pad 2: VINS+ -> +VDC
- R26 pad 1: VINS+ -> +VDC
- U11 pad 8: VINS+ -> +VDC
- U2 pad JP1_1: Net-(U2-VIN) -> +3.3V
- U7 pad 2: Net-(U7-EN) -> +VDC
- U7 pad 3: Net-(U7-EN) -> +VDC
Routing:
- net I2C1_SDA: track 0.00 -> 61.0 mm, vias 0 -> 1
- net /CORE_STM32F405/NRST: track 0.00 -> 59.9 mm, vias 0 -> 3
- net I2C1_SCL: track 0.00 -> 59.3 mm, vias 0 -> 1
- net +3.3V: track 2.26 -> 54.3 mm, vias 0 -> 25
- net IMU INT: track 0.00 -> 41.5 mm, vias 0 -> 1
- net M1_IN2: track 0.00 -> 39.7 mm, vias 0 -> 1
- net ENCODER_A_2: track 0.00 -> 37.8 mm, vias 0 -> 3
- net M1_IN1: track 0.00 -> 37.7 mm, vias 0 -> 1
- net /CORE_STM32F405/TX2: track 0.00 -> 36.9 mm
- net ALERT2_INA226: track 2.23 -> 37.6 mm, vias 0 -> 3
- net /CORE_STM32F405/RX2: track 0.00 -> 34.7 mm
- net IMU RST: track 0.00 -> 34.7 mm, vias 0 -> 1
- net SPI1_NSS: track 0.00 -> 33.4 mm, vias 0 -> 2
- net /CORE_STM32F405/TX1: track 0.00 -> 30.6 mm
- net SPI1_MISO: track 0.00 -> 29.2 mm
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- added copper zone on B.Cu, net +11.1V
- added copper zone on F.Cu, net +11.1V
- added copper zone on B.Cu, net +3.3V
- added copper zone on In2.Cu, net +3.3V
- added copper zone on F.Cu, net +3.3VA
- added copper zone on B.Cu, net +VDC
- added copper zone on F.Cu, net /CORE_STM32F405/NRST
- added copper zone on B.Cu, net /Heating_resistance/Mosfet_S
- added copper zone on B.Cu, net /Motor control/M1+
- added copper zone on F.Cu, net /Motor control/M1+
- added copper zone on B.Cu, net /Motor control/M1-
- added copper zone on F.Cu, net /Motor control/M1-
- added copper zone on B.Cu, net /Motor control/M2+
- added copper zone on F.Cu, net /Motor control/M2+
- added copper zone on B.Cu, net /Motor control/M2-
- added copper zone on F.Cu, net /Motor control/M2-
- added copper zone on F.Cu, net Net-(R2-Pad1)
- added copper zone on B.Cu, net Net-(U7-BST)
- added copper zone on B.Cu, net Net-(U7-SW)

Commit message: FINAL_V1
Parts:
- moved R18 1.29 mm to (134.3, 94.2), turned to 90 degrees
- moved C11 1.21 mm to (84.3, 104.6)
- moved C12 1.21 mm to (82.2, 104.6)
- moved C22 0.70 mm to (102.5, 84.5)
- moved R19 0.47 mm to (131.1, 94.2)
- moved C16 0.38 mm to (87.3, 82.3)
- moved C20 0.27 mm to (120.7, 85.5)
- moved C30 0.13 mm to (66.4, 101.2)
- moved LED7 0.12 mm to (136.2, 111.5)
- moved R16 0.12 mm to (132.3, 111.5)
- moved TP2 0.12 mm to (128.8, 111.5)
- moved TP3 0.12 mm to (139.7, 111.5)
Routing:
- net I2C1_SDA: track 61.0 -> 152.0 mm, vias 1 -> 3
- net ENCODER_B_1: track 4.08 -> 90.7 mm, vias 1 -> 2
- net nFAULT2: track 2.88 -> 87.4 mm, vias 1 -> 4
- net I2C1_SCL: track 59.3 -> 141.3 mm, vias 1 -> 2
- net ALERT1_INA226: track 2.09 -> 79.3 mm, vias 0 -> 1
- net PIN_MOSFET: track 13.9 -> 83.9 mm, vias 0 -> 2
- net /CORE_STM32F405/FSM_button: track 2.43 -> 69.2 mm, vias 0 -> 7
- net ENCODER_A_1: track 1.90 -> 63.3 mm, vias 1 -> 4
- net ADC1: track 7.30 -> 67.1 mm, vias 0 -> 3
- net ENCODER_B_2: track 17.2 -> 67.9 mm, vias 1 -> 4
- net +3.3V: track 54.3 -> 104.8 mm, vias 25 -> 33
- net nFAULT1: track 3.00 -> 46.4 mm, vias 1 -> 3
- net nSLEEP2: track 0.00 -> 36.4 mm, vias 0 -> 3
- net ADC2: track 7.43 -> 43.0 mm, vias 0 -> 5
- net nSLEEP1: track 1.07 -> 35.0 mm, vias 0 -> 1
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
Commit message: ESQUEMATICO
Routing:
- net I2C1_SCL: track 141.3 -> 137.0 mm
- net I2C1_SDA: track 152.0 -> 155.1 mm
- net GND: track 0.00 -> 0.94 mm, vias 0 -> 1
- net +3.3V: track 104.8 -> 105.2 mm, vias 33 -> 37
- net Net-(Q2-D): vias 3 -> 6
- net /Motor control/M2-: vias 2 -> 3

Commit message: PCB
Parts:
- moved C40 23.6 mm to (88.0, 117.9), turned to 90 degrees
- moved R21 23.0 mm to (86.4, 111.2), turned to 180 degrees
- moved U11 20.7 mm to (85.4, 114.2), turned to -90 degrees
- moved C34 18.6 mm to (66.1, 114.3), turned to 180 degrees
- moved C33 12.0 mm to (72.0, 114.3)
- moved U7 12.0 mm to (71.5, 111.2)
- moved L2 11.5 mm to (66.5, 110.8)
- moved R25 11.1 mm to (81.3, 114.1), turned to 90 degrees
- moved C35 10.7 mm to (73.5, 108.5), turned to 0 degrees
- moved C2 10.0 mm to (69.3, 106.1)
- moved R26 9.78 mm to (80.1, 109.9), turned to 0 degrees
- moved R1 8.36 mm to (67.4, 121.0)
- moved SW1 8.36 mm to (62.6, 119.2)
- moved C1 8.36 mm to (67.4, 117.3)
- moved R11 5.99 mm to (79.0, 114.1)
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Routing:
- net I2C1_SDA: track 155.1 -> 99.9 mm, vias 3 -> 2
- net /CORE_STM32F405/NRST: track 62.1 -> 34.0 mm
- net I2C1_SCL: track 137.0 -> 110.0 mm, vias 2 -> 1
- net +3.3V: track 105.2 -> 91.7 mm, vias 37 -> 51
- net /VEML 7700 Sheet/VDD_LUZ: track 11.0 -> 0.00 mm, vias 2 -> 0
- net ALERT2_INA226: track 39.8 -> 30.9 mm, vias 1 -> 0
- net +VDC: track 8.25 -> 11.7 mm, vias 1 -> 0
- net PIN_MOSFET: track 83.9 -> 80.7 mm
- net Net-(U11-VIN-): track 4.49 -> 7.41 mm
- net /CORE_STM32F405/TX2: track 38.0 -> 40.8 mm
- net GND: track 0.94 -> 2.70 mm, vias 1 -> 7
- net /CORE_STM32F405/FSM_button: track 69.2 -> 70.1 mm
- net +11.1V: vias 14 -> 19
- added copper zone on In2.Cu, net +VDC
- added copper zone on B.Cu, net GND
- removed copper zone on In2.Cu, net +3.3V
- removed copper zone on F.Cu, net /CORE_STM32F405/NRST

Commit message: FINAL
Parts:
- added G***: LOGO, LOGO, F.Cu at (67.5, 110.3)
- added G***: LOGO, LOGO, B.Cu at (107.9, 100.8)
- moved TP4 61.6 mm to (133.3, 74.4)
- moved CN3 17.2 mm to (139.0, 85.1)
- moved R19 15.8 mm to (126.1, 109.2), turned to 180 degrees
- moved R18 15.0 mm to (126.1, 106.7), turned to 180 degrees
- moved LED5 14.5 mm to (140.1, 94.0)
- moved Q1 12.4 mm to (125.2, 98.4), turned to -90 degrees
- moved R17 9.45 mm to (135.4, 94.0), turned to 0 degrees
- moved H4 5.00 mm to (141.9, 74.4)
- moved H5 5.00 mm to (141.9, 127.4)
- moved LED7 4.53 mm to (136.2, 116.0)
- moved R16 4.53 mm to (132.3, 116.0)
- moved TP2 4.53 mm to (128.8, 116.0)
- moved TP3 4.53 mm to (139.8, 116.0)
- moved C39 1.98 mm to (145.4, 118.5), turned to -90 degrees
- moved C23 1.33 mm to (123.6, 79.5)
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Connections:
- U1 pad 54: unconnected-(U1A-PD2-Pad54) -> /CORE_STM32F405/RADXA_PIN
- U3 pad : (no net) -> GND
- U4 pad : (no net) -> GND
Routing:
- net GND: track 2.70 -> 139.8 mm, vias 7 -> 68
- net /CORE_STM32F405/RADXA_PIN: track 0.00 -> 60.6 mm, vias 0 -> 3
- net ALERT1_INA226: track 79.3 -> 134.7 mm, vias 1 -> 5
- net /CORE_STM32F405/NRST: track 34.0 -> 68.2 mm, vias 3 -> 2
- net I2C1_SCL: track 110.0 -> 135.7 mm, vias 1 -> 3
- net ENCODER_B_1: track 90.7 -> 69.8 mm
- net I2C1_SDA: track 99.9 -> 120.7 mm, vias 2 -> 3
- net ALERT2_INA226: track 30.9 -> 50.7 mm, vias 0 -> 1
- net ADC2: track 43.0 -> 33.0 mm
- net IMU INT: track 49.1 -> 40.8 mm, vias 1 -> 3
- net /Heating_resistance/Mosfet_G: track 5.99 -> 13.9 mm
- net /VEML 7700 Sheet/VDD_LUZ: track 0.00 -> 7.42 mm
- net SPI1_MOSI: track 32.0 -> 26.4 mm
- net nSLEEP2: track 36.4 -> 31.8 mm
- net /CORE_STM32F405/TX2: track 40.8 -> 36.7 mm
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- added copper zone on In2.Cu, net +3.3V
- added copper zone on F.Cu, net /CORE_STM32F405/NRST
- added copper zone on F.Cu, net GND
- added copper zone on In1.Cu, net GND
- removed copper zone on F.Cu, net /Motor control/M1+
- removed copper zone on F.Cu, net /Motor control/M1-
- removed copper zone on F.Cu, net /Motor control/M2+
- removed copper zone on F.Cu, net /Motor control/M2-
Other:
- board outline added: 90 x 65 mm
- board text added: "Carlos Yujra"
- board text added: "Jair Oria"
- board text added: "Jhamir Mamani"
- board text added: "MEMBERS:"
- board text added: "Osmer Diaz"
- board text added: "Pedro Palacios"

Commit message: PCB1
Parts:
- moved H2 10.0 mm to (63.9, 64.4)
- moved H4 10.0 mm to (141.9, 64.4)
- moved J1 8.17 mm to (110.9, 64.4)
- moved J2 8.17 mm to (87.4, 64.4)
- moved C24 0.60 mm to (100.6, 79.6)
- moved C31 0.47 mm to (102.3, 79.4)
- moved C23 0.28 mm to (123.9, 79.5)
- moved C32 0.20 mm to (126.0, 79.3)
Connections:
- Q1 pad : (no net) -> GND
Routing:
- net ALERT1_INA226: track 134.7 -> 156.8 mm
- net ENCODER_B_1: track 69.8 -> 91.4 mm
- net +3.3V: track 93.5 -> 112.7 mm, vias 55 -> 43
- net ENCODER_A_2: track 41.5 -> 52.6 mm
- net ENCODER_A_1: track 63.3 -> 73.5 mm
- net ENCODER_B_2: track 70.2 -> 78.7 mm
- net GND: track 139.8 -> 136.9 mm
- net /CORE_STM32F405/NRST: track 68.2 -> 67.7 mm
- net +11.1V: vias 32 -> 31
Other:
- board size 90 x 65 mm -> 90 x 75 mm
