File: INA226_sensor_sch.kicad_sch (KiCad schematic)
At the start: 2 parts, among them U7 INA226AIDGSR, U8 INA226AIDGSR

Commit message: INA SENSOR
Parts:
- added C29, C30: 100nF, easyeda2kicad:C0402, symbol CANSAT_STM32_symbols:TCC0402X7R104J500AT
- added R2, R3: 4.7K, easyeda2kicad:R0603, symbol CANSAT_STM32_symbols:RC0603FR-074K7L
Connections:
- net GND: now reaches U8.1 (A1)
- net GND: now also U7.1 (A1), U7.2 (A0), U7.7 (GND), U8.7 (GND), C29.1, C30.1
- net +3V3: now reaches U8.2 (A0)
- net +3V3: now also U7.6 (VS+), U8.6 (VS+), C29.2, C30.2, R2.2, R3.2
- net ALERT2_INA226: now reaches U8.3 (Alert)
- net ALERT2_INA226: now also R3.1
- net I2C2_SDA: now reaches U8.4 (SDA)
- net I2C2_SDA: now also U7.4 (SDA)
- net I2C2_SCL: now reaches U8.5 (SCL)
- net I2C2_SCL: now also U7.5 (SCL)
- net VIN2+: now reaches U8.8 (VBUS)
- net ALERT1_INA226: now reaches U7.3 (Alert)
- net ALERT1_INA226: now also R2.1
- net VIN+: now reaches U7.8 (VBUS)
- no-connect marks 0 -> 4
Other:
- moved on the sheet: U7, U8

Commit message: Esquemático V1
Other:
- note added: "MEDIR CORRIENTE CON vin+ vin- BUSCAR RESISTENCIA SHUNT"
Changed lines of the file:
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@@
 	(generator_version "10.0")
 	(paper "A4")
+	(text "MEDIR CORRIENTE CON vin+ vin-\nBUSCAR RESISTENCIA SHUNT\n\n"
+		(exclude_from_sim no)
+		(at 137.16 62.23 0)
+		(effects
+			(font
+				(size 1.27 1.27)
+			)
+		)
+	)
 	(text_box "I2C Address: 0x41\n"
 		(exclude_from_sim no)

Commit message: BECERRA
Other:
- moved on the sheet: C29, C30, R2, R3, U7, U8

Commit message: feat: [solución de rules checker]
Connections:
- net VIN+: no longer names the net of U7.8 (VBUS)
Changed lines of the file:
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@@
 	(wire
 		(pts
-			(xy 58.42 83.82) (xy 58.42 87.63)
+			(xy 130.81 74.93) (xy 134.62 74.93)
 		)
 		(stroke
@@
 	(wire
 		(pts
-			(xy 58.42 71.12) (xy 58.42 73.66)
+			(xy 58.42 83.82) (xy 58.42 87.63)
 		)
 		(stroke
@@
 	(wire
 		(pts
-			(xy 196.85 77.47) (xy 198.12 77.47)
+			(xy 58.42 71.12) (xy 58.42 73.66)
 		)
 		(stroke
@@
 	(wire
 		(pts
-			(xy 153.67 97.79) (xy 153.67 100.33)
+			(xy 196.85 77.47) (xy 198.12 77.47)
 		)
 		(stroke
@@
 	(wire
 		(pts
-			(xy 85.09 99.06) (xy 85.09 101.6)
+			(xy 153.67 97.79) (xy 153.67 100.33)
 		)
 		(stroke
@@
 	(wire
 		(pts
-			(xy 130.81 74.93) (xy 132.08 74.93)
+			(xy 85.09 99.06) (xy 85.09 101.6)
 		)
 		(stroke
@@
 	)
 	(symbol
+		(lib_name "+3V3_1")
 		(lib_id "power:+3V3")
-		(at 132.08 74.93 270)
+		(at 134.62 74.93 270)
 		(mirror x)
 		(unit 1)
@@
 		(fields_autoplaced yes)
 		(property "Reference" "#PWR093"
-			(at 128.27 74.93 0)
+			(at 130.81 74.93 0)
 			(hide yes)
 			(show_name no)
@@
 		)
 		(property "Value" "VIN+"
-			(at 135.89 74.9299 90)
+			(at 138.43 74.9299 90)
 			(show_name no)
 			(do_not_autoplace no)
@@
 		)
 		(property "Footprint" ""
-			(at 132.08 74.93 0)
+			(at 134.62 74.93 0)
 			(hide yes)
 			(show_name no)
@@
 		)
 		(property "Datasheet" ""
-			(at 132.08 74.93 0)
+			(at 134.62 74.93 0)
 			(hide yes)
 			(show_name no)
@@
 		)
 		(property "Description" "Power symbol creates a global label with name \"+3V3\""
-			(at 132.08 74.93 0)
+			(at 134.62 74.93 0)
 			(hide yes)
 			(show_name no)
@@
 	)
 	(symbol
+		(lib_name "INA226AIDGSR_1")
 		(lib_id "CANSAT_STM32_symbols:INA226AIDGSR")
 		(at 184.15 74.93 0)

Commit message: Cantidad de errores en la PCB: 29
Parts:
- C29, C30: footprint easyeda2kicad:C0402 -> ARLISS-footprints:C0402
- R3: footprint easyeda2kicad:R0603 -> ARLISS-footprints:R0603
Changed lines of the file:
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@@
 			)
 		)
-		(property "Footprint" "easyeda2kicad:R0603"
+		(property "Footprint" "ARLISS-footprints:R0603"
 			(at 228.6 78.74 0)
 			(hide yes)
@@
 			)
 		)
-		(property "Footprint" "easyeda2kicad:C0402"
+		(property "Footprint" "ARLISS-footprints:C0402"
 			(at 92.71 93.98 0)
 			(hide yes)
@@
 			)
 		)
-		(property "Footprint" "easyeda2kicad:C0402"
+		(property "Footprint" "ARLISS-footprints:C0402"
 			(at 161.29 92.71 0)
 			(hide yes)

Commit message: Cantidad de errores de la placa: 05
Parts:
- R2: footprint easyeda2kicad:R0603 -> ARLISS-footprints:R0603
- U7, U8: footprint easyeda2kicad:MSOP-10_L3.0-W3.0-P0.50-LS5.0-BL -> ARLISS-footprints:MSOP-10_L3.0-W3.0-P0.50-LS5.0-BL
Changed lines of the file:
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@@
 			)
 		)
-		(property "Footprint" "easyeda2kicad:R0603"
+		(property "Footprint" "ARLISS-footprints:R0603"
 			(at 66.04 78.74 0)
 			(hide yes)
@@
 			)
 		)
-		(property "Footprint" "easyeda2kicad:MSOP-10_L3.0-W3.0-P0.50-LS5.0-BL"
+		(property "Footprint" "ARLISS-footprints:MSOP-10_L3.0-W3.0-P0.50-LS5.0-BL"
 			(at 184.15 87.63 0)
 			(hide yes)
@@
 			)
 		)
-		(property "Footprint" "easyeda2kicad:MSOP-10_L3.0-W3.0-P0.50-LS5.0-BL"
+		(property "Footprint" "ARLISS-footprints:MSOP-10_L3.0-W3.0-P0.50-LS5.0-BL"
 			(at 118.11 87.63 0)
 			(hide yes)

Commit message: PCB ordenada V1
Connections:
- net I2C2_SCL renamed I2C1_SCL
- net I2C2_SDA renamed I2C1_SDA
Changed lines of the file:
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@@
 		)
 	)
-	(global_label "I2C2_SCL"
+	(global_label "I2C1_SCL"
 		(shape input)
 		(at 168.91 80.01 180)
@@
 		)
 	)
-	(global_label "I2C2_SDA"
+	(global_label "I2C1_SDA"
 		(shape input)
 		(at 168.91 77.47 180)
@@
 		)
 	)
-	(global_label "I2C2_SDA"
+	(global_label "I2C1_SDA"
 		(shape input)
 		(at 102.87 77.47 180)
@@
 		)
 	)
-	(global_label "I2C2_SCL"
+	(global_label "I2C1_SCL"
 		(shape input)
 		(at 102.87 80.01 180)

Commit message: Primer Ruteo de PCB
Parts:
- C29, C30: footprint ARLISS-footprints:C0402 -> Capacitor_SMD:C_0402_1005Metric_Pad0.74x0.62mm_HandSolder
Changed lines of the file:
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@@
 			)
 		)
-		(property "Footprint" "ARLISS-footprints:C0402"
+		(property "Footprint" "Capacitor_SMD:C_0402_1005Metric_Pad0.74x0.62mm_HandSolder"
 			(at 92.71 93.98 0)
 			(hide yes)
@@
 			)
 		)
-		(property "Footprint" "ARLISS-footprints:C0402"
+		(property "Footprint" "Capacitor_SMD:C_0402_1005Metric_Pad0.74x0.62mm_HandSolder"
 			(at 161.29 92.71 0)
 			(hide yes)
