File: ARLISS_STM32_2026.kicad_sch (KiCad schematic)
At the start: 0 parts

Commit message: Arreglos de esquemático
Parts:
- added H1, H2, H3, H4, H5, H6: MountingHole, MountingHole:MountingHole_3.2mm_M3_ISO14580_Pad, symbol Mechanical:MountingHole
Other:
- sheet Alimentacion: file untitled.kicad_sch -> POWER_V.kicad_sch

Commit message: Arreglando footprints
Parts:
- H1, H2, H3, H4, H5, H6: now in the parts list
Other:
- company: (none) -> TOMEK TEAM
- title: (none) -> ARLISS STM32 BOARD
Changed lines of the file:
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@@
 	(generator_version "10.0")
 	(paper "A4")
+	(title_block
+		(title "ARLISS STM32 BOARD")
+		(date "2026-06-21")
+		(rev "A")
+		(company "TOMEK TEAM")
+		(comment 1 "https://github.com/JosephPalacios-so/CANSAT_ARLISS.git")
+	)
 	(text_box "SPI_1 INTERFACE"
 		(exclude_from_sim no)
@@
 		(body_style 1)
 		(exclude_from_sim no)
-		(in_bom no)
+		(in_bom yes)
 		(on_board yes)
 		(in_pos_files yes)
@@
 		(body_style 1)
 		(exclude_from_sim no)
-		(in_bom no)
+		(in_bom yes)
 		(on_board yes)
 		(in_pos_files yes)
@@
 		(body_style 1)
 		(exclude_from_sim no)
-		(in_bom no)
+		(in_bom yes)
 		(on_board yes)
 		(in_pos_files yes)
@@
 		(body_style 1)
 		(exclude_from_sim no)
-		(in_bom no)
+		(in_bom yes)
 		(on_board yes)
 		(in_pos_files yes)
@@
 		(body_style 1)
 		(exclude_from_sim no)
-		(in_bom no)
+		(in_bom yes)
 		(on_board yes)
 		(in_pos_files yes)
@@
 		(body_style 1)
 		(exclude_from_sim no)
-		(in_bom no)
-		(on_board yes)
-		(in_pos_files yes)
+		(in_bom yes)
+		(on_board yes)
+		(in_pos_files yes)
