File: ADXL375.kicad_sch (KiCad schematic)
At the start: 5 parts, among them U6 ADXL372BCCZ-RL

Commit message: Arreglos de esquemático
Parts:
- L1: footprint ARLISS-footprints:L0402 -> Inductor_SMD:L_0402_1005Metric_Pad0.77x0.64mm_HandSolder
Changed lines of the file:
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@@
 			)
 		)
-		(property "Footprint" "ARLISS-footprints:L0402"
+		(property "Footprint" "Inductor_SMD:L_0402_1005Metric_Pad0.77x0.64mm_HandSolder"
 			(at 228.6 101.6 0)
 			(hide yes)

Commit message: Arreglando footprints
Parts:
- C36: renamed from C7; footprint Capacitor_SMD:C_0402_1005Metric_Pad0.74x0.62mm_HandSolder -> Capacitor_SMD:C_0603_1608Metric_Pad1.08x0.95mm_HandSolder; Manufacturer CCTC(三环) -> (none)
- C37: renamed from C27; footprint Capacitor_SMD:C_0402_1005Metric_Pad0.74x0.62mm_HandSolder -> Capacitor_SMD:C_0603_1608Metric_Pad1.08x0.95mm_HandSolder; Manufacturer CCTC(三环) -> (none)
- C38: renamed from C28; Manufacturer Kyocera AVX -> (none)
- L3: renamed from L1; Manufacturer FH(风华) -> (none)
- U9: renamed from U6; Manufacturer ADI(亚德诺) -> (none)
Other:
- company: (none) -> TOMEK TEAM
Changed lines of the file:
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@@
 	(generator_version "10.0")
 	(paper "A4")
+	(title_block
+		(company "TOMEK TEAM")
+	)
 	(junction
 		(at 128.27 88.9)
@@
 		(dnp no)
 		(fields_autoplaced yes)
-		(property "Reference" "C7"
+		(property "Reference" "C36"
 			(at 132.08 95.2499 90)
 			(show_name no)
@@
 			)
 		)
-		(property "Footprint" "Capacitor_SMD:C_0402_1005Metric_Pad0.74x0.62mm_HandSolder"
+		(property "Footprint" "Capacitor_SMD:C_0603_1608Metric_Pad1.08x0.95mm_HandSolder"
 			(at 135.89 96.52 0)
 			(hide yes)
@@
 			)
 		)
-		(property "Manufacturer" "CCTC(三环)"
-			(at 140.97 96.52 0)
-			(hide yes)
-			(show_name no)
-			(do_not_autoplace no)
-			(effects
-				(font
-					(size 1.27 1.27)
-				)
-			)
-		)
 		(property "MPN" "TCC0402X7R104J500AT"
 			(at 143.51 96.52 0)
@@
 			(project "ARLISS_STM32_2026"
 				(path "/9719ea46-14c4-4409-9c57-49dd5454c03f/5dc414a7-f6ea-4307-9bff-662079fd3375"
-					(reference "C7")
+					(reference "C36")
 					(unit 1)
 				)
@@
 		(dnp no)
 		(fields_autoplaced yes)
-		(property "Reference" "#PWR066"
+		(property "Reference" "#PWR0105"
 			(at 128.27 110.49 0)
 			(hide yes)
@@
 			(project "ARLISS_STM32_2026"
 				(path "/9719ea46-14c4-4409-9c57-49dd5454c03f/5dc414a7-f6ea-4307-9bff-662079fd3375"
-					(reference "#PWR066")
+					(reference "#PWR0105")
 					(unit 1)
 				)
@@
 		(dnp no)
 		(fields_autoplaced yes)
-		(property "Reference" "C27"
+		(property "Reference" "C37"
 			(at 209.55 100.3299 90)
 			(show_name no)
@@
 			)
 		)
-		(property "Footprint" "Capacitor_SMD:C_0402_1005Metric_Pad0.74x0.62mm_HandSolder"
+		(property "Footprint" "Capacitor_SMD:C_0603_1608Metric_Pad1.08x0.95mm_HandSolder"
 			(at 213.36 101.6 0)
 			(hide yes)
@@
 			)
 		)
-		(property "Manufacturer" "CCTC(三环)"
-			(at 218.44 101.6 0)
-			(hide yes)
-			(show_name no)
-			(do_not_autoplace no)
-			(effects
-				(font
-					(size 1.27 1.27)
-				)
-			)
-		)
 		(property "MPN" "TCC0402X7R104J500AT"
 			(at 220.98 101.6 0)
@@
 			(project "ARLISS_STM32_2026"
 				(path "/9719ea46-14c4-4409-9c57-49dd5454c03f/5dc414a7-f6ea-4307-9bff-662079fd3375"
-					(reference "C27")
+					(reference "C37")
 					(unit 1)
 				)
@@
 		(dnp no)
 		(fields_autoplaced yes)
-		(property "Reference" "#PWR065"
+		(property "Reference" "#PWR0108"
 			(at 238.76 97.79 0)
 			(hide yes)
@@
 			(project "ARLISS_STM32_2026"
 				(path "/9719ea46-14c4-4409-9c57-49dd5454c03f/5dc414a7-f6ea-4307-9bff-662079fd3375"
-					(reference "#PWR065")
+					(reference "#PWR0108")
 					(unit 1)
 				)
@@
 		(dnp no)
 		(fields_autoplaced yes)
-		(property "Reference" "U6"
+		(property "Reference" "U9"
 			(at 171.45 81.28 0)
 			(show_name no)
@@
 			)
 		)
-		(property "Manufacturer" "ADI(亚德诺)"
-			(at 171.45 119.38 0)
-			(hide yes)
-			(show_name no)
-			(do_not_autoplace no)
-			(effects
-				(font
-					(size 1.27 1.27)
-				)
-			)
-		)
 		(property "MPN" "ADXL372BCCZ-RL"
 			(at 171.45 121.92 0)
@@
 			(project "ARLISS_STM32_2026"
 				(path "/9719ea46-14c4-4409-9c57-49dd5454c03f/5dc414a7-f6ea-4307-9bff-662079fd3375"
-					(reference "U6")
+					(reference "U9")
 					(unit 1)
 				)
@@
 		(dnp no)
 		(fields_autoplaced yes)
-		(property "Reference" "#PWR067"
+		(property "Reference" "#PWR0107"
 			(at 205.74 115.57 0)
 			(hide yes)
@@
 			(project "ARLISS_STM32_2026"
 				(path "/9719ea46-14c4-4409-9c57-49dd5454c03f/5dc414a7-f6ea-4307-9bff-662079fd3375"
-					(reference "#PWR067")
+					(reference "#PWR0107")
 					(unit 1)
 				)
@@
 		(dnp no)
 		(fields_autoplaced yes)
-		(property "Reference" "L1"
+		(property "Reference" "L3"
 			(at 228.57 87.63 0)
 			(show_name no)
@@
 			)
 		)
-		(property "Manufacturer" "FH(风华)"
-			(at 228.6 106.68 0)
-			(hide yes)
-			(show_name no)
-			(do_not_autoplace no)
-			(effects
-				(font
-					(size 1.27 1.27)
-				)
-			)
-		)
 		(property "MPN" "CBG100505U000T"
 			(at 228.6 109.22 0)
@@
 			(project "ARLISS_STM32_2026"
 				(path "/9719ea46-14c4-4409-9c57-49dd5454c03f/5dc414a7-f6ea-4307-9bff-662079fd3375"
-					(reference "L1")
+					(reference "L3")
 					(unit 1)
 				)
@@
 		(in_pos_files yes)
 		(dnp no)
-		(property "Reference" "#PWR041"
+		(property "Reference" "#PWR0104"
 			(at 120.65 92.71 0)
 			(hide yes)
@@
 			(project "ARLISS_STM32_2026"
 				(path "/9719ea46-14c4-4409-9c57-49dd5454c03f/5dc414a7-f6ea-4307-9bff-662079fd3375"
-					(reference "#PWR041")
+					(reference "#PWR0104")
 					(unit 1)
 				)
@@
 		(dnp no)
 		(fields_autoplaced yes)
-		(property "Reference" "#PWR034"
+		(property "Reference" "#PWR0106"
 			(at 199.39 88.9 0)
 			(hide yes)
@@
 			(project "ARLISS_STM32_2026"
 				(path "/9719ea46-14c4-4409-9c57-49dd5454c03f/5dc414a7-f6ea-4307-9bff-662079fd3375"
-					(reference "#PWR034")
+					(reference "#PWR0106")
 					(unit 1)
 				)
@@
 		(dnp no)
 		(fields_autoplaced yes)
-		(property "Reference" "C28"
+		(property "Reference" "C38"
 			(at 222.25 99.6949 90)
 			(show_name no)
@@
 			)
 		)
-		(property "Manufacturer" "Kyocera AVX"
-			(at 231.14 101.6 0)
-			(hide yes)
-			(show_name no)
-			(do_not_autoplace no)
-			(effects
-				(font
-					(size 1.27 1.27)
-				)
-			)
-		)
 		(property "MPN" "TAJB105K035RNJ"
 			(at 233.68 101.6 0)
@@
 			(project "ARLISS_STM32_2026"
 				(path "/9719ea46-14c4-4409-9c57-49dd5454c03f/5dc414a7-f6ea-4307-9bff-662079fd3375"
-					(reference "C28")
+					(reference "C38")
 					(unit 1)
 				)

Commit message: Todo antes de PCB
Parts:
- L3: value 0R 100Mhz -> 90R 100Mhz; footprint Inductor_SMD:L_0402_1005Metric_Pad0.77x0.64mm_HandSolder -> Inductor_SMD:L_0603_1608Metric_Pad1.05x0.95mm_HandSolder; LCSC Part C139137 -> C50325905; MPN CBG100505U000T -> APBD1608-900WTD12
Connections:
- net SPI2_CSK renamed SPI2_SCLK
- net SPI2_NSS renamed SPI2_CS
Changed lines of the file:
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@@
 		)
 	)
-	(global_label "SPI2_NSS"
+	(global_label "SPI2_CS"
 		(shape input)
 		(at 153.67 106.68 180)
@@
 		)
 		(property "Intersheetrefs" "${INTERSHEET_REFS}"
-			(at 141.6739 106.68 0)
+			(at 142.9439 106.68 0)
 			(hide yes)
 			(show_name no)
@@
 		)
 	)
-	(global_label "SPI2_CSK"
+	(global_label "SPI2_SCLK"
 		(shape input)
 		(at 153.67 96.52 180)
@@
 		)
 		(property "Intersheetrefs" "${INTERSHEET_REFS}"
-			(at 141.6739 96.52 0)
+			(at 140.6458 96.52 0)
 			(hide yes)
 			(show_name no)
@@
 			)
 		)
-		(property "Value" "0R 100Mhz"
+		(property "Value" "90R 100Mhz"
 			(at 228.57 90.17 0)
 			(show_name no)
@@
 			)
 		)
-		(property "Footprint" "Inductor_SMD:L_0402_1005Metric_Pad0.77x0.64mm_HandSolder"
+		(property "Footprint" "Inductor_SMD:L_0603_1608Metric_Pad1.05x0.95mm_HandSolder"
 			(at 228.6 101.6 0)
 			(hide yes)
@@
 			)
 		)
-		(property "Datasheet" "https://lcsc.com/product-detail/Ferrite-Beads-And-Chips_0R-25_C139137.html"
+		(property "Datasheet" "https://www.lcsc.com/datasheet/C50325905.pdf?spm=wm.sxq.inf.ggs___wm.fly.bg.2.xh&lcsc_vid=E1NWVQUCRlhbBlQCFAQIVQJXQ1UKV1AATgdWXgAERFExVlNeRVBaX1ZST1RWXjsOAxUeFF5JWBYZEEoKFBINSQcJGk4dAgUUFAk%3D"
 			(at 228.6 104.14 0)
 			(hide yes)
@@
 			)
 		)
-		(property "MPN" "CBG100505U000T"
+		(property "MPN" "APBD1608-900WTD12"
 			(at 228.6 109.22 0)
 			(hide yes)
@@
 			)
 		)
-		(property "LCSC Part" "C139137"
+		(property "LCSC Part" "C50325905"
 			(at 228.6 111.76 0)
 			(hide yes)
