File: EsquemáticoSTM32F405.kicad_sch (KiCad schematic)
At the start: 30 parts, among them P1 PZ254R-12-8P, SW3 EVQPLMA15, SW4 EVQPLMA15, U4 STM32F405RGT6, X1 32.768kHz 7pF SMD, X2 8Mhz 10pF

Commit message: Arreglando footprints
Parts:
- C1: renamed from C22; footprint Capacitor_SMD:C_0402_1005Metric_Pad0.74x0.62mm_HandSolder -> Capacitor_SMD:C_0603_1608Metric_Pad1.08x0.95mm_HandSolder; Manufacturer CCTC(三环) -> (none)
- C10: renamed from C17; footprint Capacitor_SMD:C_0402_1005Metric_Pad0.74x0.62mm_HandSolder -> Capacitor_SMD:C_0603_1608Metric_Pad1.08x0.95mm_HandSolder; Manufacturer CCTC(三环) -> (none)
- C11: renamed from C13; footprint Capacitor_SMD:C_0402_1005Metric_Pad0.74x0.62mm_HandSolder -> Capacitor_SMD:C_0603_1608Metric_Pad1.08x0.95mm_HandSolder; Manufacturer YAGEO(国巨) -> (none)
- C12: footprint Capacitor_SMD:C_0402_1005Metric_Pad0.74x0.62mm_HandSolder -> Capacitor_SMD:C_0603_1608Metric_Pad1.08x0.95mm_HandSolder; Manufacturer YAGEO(国巨) -> (none)
- C13: renamed from C18; footprint Capacitor_SMD:C_0402_1005Metric_Pad0.74x0.62mm_HandSolder -> Capacitor_SMD:C_0603_1608Metric_Pad1.08x0.95mm_HandSolder
- C14: renamed from C19; footprint Capacitor_SMD:C_0402_1005Metric_Pad0.74x0.62mm_HandSolder -> Capacitor_SMD:C_0603_1608Metric_Pad1.08x0.95mm_HandSolder; Manufacturer HRE(芯声) -> (none)
- C2: renamed from C26; footprint Capacitor_SMD:C_0402_1005Metric_Pad0.74x0.62mm_HandSolder -> Capacitor_SMD:C_0603_1608Metric_Pad1.08x0.95mm_HandSolder; Manufacturer CCTC(三环) -> (none)
- C3: renamed from C23; footprint Capacitor_SMD:C_0402_1005Metric_Pad0.74x0.62mm_HandSolder -> Capacitor_SMD:C_0603_1608Metric_Pad1.08x0.95mm_HandSolder; Manufacturer YAGEO(国巨) -> (none)
- C4: renamed from C11; footprint Capacitor_SMD:C_0402_1005Metric_Pad0.74x0.62mm_HandSolder -> Capacitor_SMD:C_0603_1608Metric_Pad1.08x0.95mm_HandSolder; Manufacturer YAGEO(国巨) -> (none)
- C5: renamed from C20; footprint Capacitor_SMD:C_0402_1005Metric_Pad0.74x0.62mm_HandSolder -> Capacitor_SMD:C_0603_1608Metric_Pad1.08x0.95mm_HandSolder; Manufacturer muRata(村田) -> (none)
- C6: renamed from C21; footprint Capacitor_SMD:C_0402_1005Metric_Pad0.74x0.62mm_HandSolder -> Capacitor_SMD:C_0603_1608Metric_Pad1.08x0.95mm_HandSolder; Manufacturer muRata(村田) -> (none)
- C7: renamed from C16; footprint Capacitor_SMD:C_0402_1005Metric_Pad0.74x0.62mm_HandSolder -> Capacitor_SMD:C_0603_1608Metric_Pad1.08x0.95mm_HandSolder; Manufacturer CCTC(三环) -> (none)
- C8: renamed from C14; footprint Capacitor_SMD:C_0402_1005Metric_Pad0.74x0.62mm_HandSolder -> Capacitor_SMD:C_0603_1608Metric_Pad1.08x0.95mm_HandSolder; Manufacturer CCTC(三环) -> (none)
- C9: renamed from C15; footprint Capacitor_SMD:C_0402_1005Metric_Pad0.74x0.62mm_HandSolder -> Capacitor_SMD:C_0603_1608Metric_Pad1.08x0.95mm_HandSolder; Manufacturer CCTC(三环) -> (none)
- L1: renamed from L3; Manufacturer muRata(村田) -> (none)
- LED1: renamed from LED3; Manufacturer ARKLED(方舟) -> (none)
- P1: Manufacturer XFCN(兴飞) -> (none)
- R1: renamed from R11; Manufacturer YAGEO(国巨) -> (none)
- R2: renamed from R12; Manufacturer YAGEO(国巨) -> (none)
- R3: renamed from R10; Manufacturer YAGEO(国巨) -> (none)
- R4: renamed from R13; Manufacturer YAGEO(国巨) -> (none)
- R7: renamed from R4; Manufacturer YAGEO(国巨) -> (none)
- R8: renamed from R5; Manufacturer YAGEO(国巨) -> (none)
- SW1: renamed from SW4; Manufacturer PANASONIC(松下) -> (none)
- SW2: renamed from SW3; Manufacturer PANASONIC(松下) -> (none)
- U1: renamed from U4; Manufacturer ST(意法半导体) -> (none)
- X1: Manufacturer EPSON(爱普生) -> (none)
- X2: Manufacturer 同晶 -> (none)
- renumbered R7 to R5, R8 to R6
Other:
- company: (none) -> TOMEK TEAM

Commit message: Todo antes de PCB
Parts:
- added CN3: 436500300, ARLISS-footprints:CONN-TH_3P-436500300, symbol CANSAT_STM32_symbols:436500300
- L1: footprint Inductor_SMD:L_0402_1005Metric_Pad0.77x0.64mm_HandSolder -> Inductor_SMD:L_0603_1608Metric_Pad1.05x0.95mm_HandSolder
Connections:
- net GND: now also CN3.3
- net RADXA_RX2 renamed RX2
- net RX2: now also CN3.2
- net RADXA_TX2 renamed TX2
- net TX2: now also CN3.1
- net SPI1_SCK renamed SPI1_SCLK
- net SPI2_CSK renamed SPI2_SCLK
- net SPI2_NSS renamed SPI2_CS
Other:
- moved on the sheet: C11, C12, R7, R8, X2
