File: EsquemáticoSTM32F405.kicad_sch (KiCad schematic)
At the start: 31 parts, among them CN3 436500300, P1 PZ254R-12-8P, SW1 EVQPLMA15, SW2 EVQPLMA15, U1 STM32F405RGT6, X1 32.768kHz 7pF SMD, X2 8Mhz 10pF

Commit message: C14 y C1,C2,... modificados
Parts:
- C1, C10, C2, C7, C8, C9: LCSC Part C5448844 -> C282518
- C14: LCSC Part C6119811 -> C559769

Commit message: PCB Solucionado
Parts:
- C11, C12: LCSC Part C513681 -> C309467
- C13: LCSC Part (none) -> C100042
- C3: value 7p -> 7pF; LCSC Part C260628 -> C519115
- C4: LCSC Part C260628 -> C519115
- C5, C6: LCSC Part C2999759 -> C86018
- L1: LCSC Part C76889 -> C307758
Changed lines of the file:
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@@
 			)
 		)
-		(property "Datasheet" "https://www.lcsc.com/datasheet/C282518.pdf?spm=wm.sxq.inf.ggs___wm.fly.bg.0.cbh&lcsc_vid=FVBZXlJVElFWAVdTTgAPVAcHR1hXAlIFT1cMUAFWQVYxVlNeRFBfVlJeQ1VXXzsOAxUeFF5JWBYZEEoKFBINSQcJGk4NBhADEA4cHktXRlVcSQwSGg0%3D"
+		(property "Datasheet" "https://www.lcsc.com/datasheet/C282518.pdf"
 			(at 340.36 58.42 0)
 			(hide yes)
@@
 			)
 		)
-		(property "Datasheet" "https://lcsc.com/product-detail/Multilayer-Ceramic-Capacitors-MLCC-SMD-SMT_YAGEO-CC0402FRNPO9BN100_C513681.html"
+		(property "Datasheet" "https://www.lcsc.com/datasheet/C309467.pdf"
 			(at 353.06 217.17 0)
 			(hide yes)
@@
 			)
 		)
-		(property "LCSC Part" "C513681"
+		(property "LCSC Part" "C309467"
 			(at 353.06 224.79 0)
 			(hide yes)
@@
 			)
 		)
-		(property "Datasheet" "https://www.lcsc.com/datasheet/C559769.pdf?spm=wm.sxq.inf.ggs___wm.fly.bg.0.xh&lcsc_vid=FVBZXlJVElFWAVdTTgAPVAcHR1hXAlIFT1cMUAFWQVYxVlNeRFBcX1JXQ1BZXzsOAxUeFF5JWBYZEEoKFBINSQcJGk4%3D"
+		(property "Datasheet" "https://www.lcsc.com/datasheet/C559769.pdf"
 			(at 403.86 57.15 0)
 			(hide yes)
@@
 			)
 		)
-		(property "Datasheet" "https://www.lcsc.com/datasheet/C282518.pdf?spm=wm.sxq.inf.ggs___wm.fly.bg.0.cbh&lcsc_vid=FVBZXlJVElFWAVdTTgAPVAcHR1hXAlIFT1cMUAFWQVYxVlNeRFBfVlJeQ1VXXzsOAxUeFF5JWBYZEEoKFBINSQcJGk4NBhADEA4cHktXRlVcSQwSGg0%3D"
+		(property "Datasheet" "https://www.lcsc.com/datasheet/C282518.pdf"
 			(at 320.04 58.42 0)
 			(hide yes)
@@
 			)
 		)
-		(property "Datasheet" "https://www.lcsc.com/datasheet/C282518.pdf?spm=wm.sxq.inf.ggs___wm.fly.bg.0.cbh&lcsc_vid=FVBZXlJVElFWAVdTTgAPVAcHR1hXAlIFT1cMUAFWQVYxVlNeRFBfVlJeQ1VXXzsOAxUeFF5JWBYZEEoKFBINSQcJGk4NBhADEA4cHktXRlVcSQwSGg0%3D"
+		(property "Datasheet" "https://www.lcsc.com/datasheet/C282518.pdf"
 			(at 49.53 81.28 0)
 			(hide yes)
@@
 			)
 		)
-		(property "Datasheet" "https://www.lcsc.com/datasheet/C282518.pdf?spm=wm.sxq.inf.ggs___wm.fly.bg.0.cbh&lcsc_vid=FVBZXlJVElFWAVdTTgAPVAcHR1hXAlIFT1cMUAFWQVYxVlNeRFBfVlJeQ1VXXzsOAxUeFF5JWBYZEEoKFBINSQcJGk4NBhADEA4cHktXRlVcSQwSGg0%3D"
+		(property "Datasheet" "https://www.lcsc.com/datasheet/C282518.pdf"
 			(at 330.2 58.42 0)
 			(hide yes)
@@
 			)
 		)
-		(property "Datasheet" "https://www.lcsc.com/datasheet/C2999759.pdf"
+		(property "Datasheet" "https://www.lcsc.com/datasheet/C86018.pdf"
 			(at 334.01 218.44 0)
 			(hide yes)
@@
 			)
 		)
-		(property "LCSC Part" "C2999759"
+		(property "LCSC Part" "C86018"
 			(at 341.63 218.44 0)
 			(hide yes)
@@
 			)
 		)
-		(property "Datasheet" "https://www.lcsc.com/datasheet/C282518.pdf?spm=wm.sxq.inf.ggs___wm.fly.bg.0.cbh&lcsc_vid=FVBZXlJVElFWAVdTTgAPVAcHR1hXAlIFT1cMUAFWQVYxVlNeRFBfVlJeQ1VXXzsOAxUeFF5JWBYZEEoKFBINSQcJGk4NBhADEA4cHktXRlVcSQwSGg0%3D"
+		(property "Datasheet" "https://www.lcsc.com/datasheet/C282518.pdf"
 			(at 179.07 72.39 0)
 			(hide yes)
@@
 			)
 		)
-		(property "Datasheet" "https://lcsc.com/product-detail/_YAGEO-CC0402CRNPO9BN7R0_C260628.html"
+		(property "Datasheet" "https://www.lcsc.com/datasheet/C519115.pdf"
 			(at 243.84 234.95 0)
 			(hide yes)
@@
 			)
 		)
-		(property "LCSC Part" "C260628"
+		(property "LCSC Part" "C519115"
 			(at 251.46 234.95 0)
 			(hide yes)
@@
 			)
 		)
-		(property "Datasheet" "https://lcsc.com/product-detail/Ferrite-Beads-And-Chips_muRata_BLM15HG102SN1D_1KR-at100MHz_C76889.html"
+		(property "Datasheet" "https://www.lcsc.com/datasheet/C307758.pdf"
 			(at 370.84 59.69 0)
 			(hide yes)
@@
 			)
 		)
-		(property "LCSC Part" "C76889"
+		(property "LCSC Part" "C307758"
 			(at 370.84 67.31 0)
 			(hide yes)
@@
 			)
 		)
-		(property "Value" "7p"
+		(property "Value" "7pF"
 			(at 237.49 210.8199 90)
 			(show_name no)
@@
 			)
 		)
-		(property "Datasheet" "https://lcsc.com/product-detail/_YAGEO-CC0402CRNPO9BN7R0_C260628.html"
+		(property "Datasheet" "https://www.lcsc.com/datasheet/C519115.pdf"
 			(at 243.84 209.55 0)
 			(hide yes)
@@
 			)
 		)
-		(property "LCSC Part" "C260628"
+		(property "LCSC Part" "C519115"
 			(at 251.46 209.55 0)
 			(hide yes)
@@
 			)
 		)
-		(property "Datasheet" ""
+		(property "Datasheet" "https://www.lcsc.com/datasheet/C100042.pdf"
 			(at 381 57.15 0)
 			(hide yes)
@@
 			)
 		)
+		(property "LCSC Part" "C100042"
+			(at 381 57.15 0)
+			(hide yes)
+			(show_name no)
+			(do_not_autoplace no)
+			(effects
+				(font
+					(size 1.27 1.27)
+				)
+			)
+		)
 		(pin "2"
 		)
@@
 			)
 		)
-		(property "Datasheet" "https://www.lcsc.com/datasheet/C282518.pdf?spm=wm.sxq.inf.ggs___wm.fly.bg.0.cbh&lcsc_vid=FVBZXlJVElFWAVdTTgAPVAcHR1hXAlIFT1cMUAFWQVYxVlNeRFBfVlJeQ1VXXzsOAxUeFF5JWBYZEEoKFBINSQcJGk4NBhADEA4cHktXRlVcSQwSGg0%3D"
+		(property "Datasheet" "https://www.lcsc.com/datasheet/C282518.pdf"
 			(at 350.52 58.42 0)
 			(hide yes)
@@
 			)
 		)
-		(property "Datasheet" "https://lcsc.com/product-detail/Multilayer-Ceramic-Capacitors-MLCC-SMD-SMT_YAGEO-CC0402FRNPO9BN100_C513681.html"
+		(property "Datasheet" "https://www.lcsc.com/datasheet/C309467.pdf"
 			(at 356.87 175.26 0)
 			(hide yes)
@@
 			)
 		)
-		(property "LCSC Part" "C513681"
+		(property "LCSC Part" "C309467"
 			(at 364.49 175.26 0)
 			(hide yes)
@@
 			)
 		)
-		(property "Datasheet" "https://www.lcsc.com/datasheet/C2999759.pdf"
+		(property "Datasheet" "https://www.lcsc.com/datasheet/C86018.pdf"
 			(at 320.04 218.44 0)
 			(hide yes)
@@
 			)
 		)
-		(property "LCSC Part" "C2999759"
+		(property "LCSC Part" "C86018"
 			(at 327.66 218.44 0)
 			(hide yes)

Commit message: Avance 02/08
Parts:
- removed CN3: 436500300, ARLISS-footprints:CONN-TH_3P-436500300, symbol CANSAT_STM32_symbols:436500300
- added CN4: 0430450400, ARLISS-footprints:CONN-TH_0430450400, symbol CANSAT_STM32_symbols:0430450400
- C13: LCSC Part C100042 -> C115056
Connections:
- net GND: now also CN4.1, CN4.2
- net RX2: now also CN4.3
- net TX2: now also CN4.4

Commit message: FINAL SCHEMATIC
Parts:
- removed C2: 100nF, Capacitor_SMD:C_0603_1608Metric_Pad1.08x0.95mm_HandSolder, symbol CANSAT_STM32_symbols:TCC0402X7R104J500AT
- removed R5: 10k, Resistor_SMD:R_0603_1608Metric_Pad0.98x0.95mm_HandSolder, symbol Device:R_Small
- added C28: 1uF, Capacitor_SMD:C_0603_1608Metric_Pad1.08x0.95mm_HandSolder, symbol CANSAT_STM32_symbols:CGA0402X5R105K500GT
- added R5: 10K, Resistor_SMD:R_0603_1608Metric_Pad0.98x0.95mm_HandSolder, symbol CANSAT_STM32_symbols:RC0603FR-7W10KL
- C13: LCSC C5448827 -> C85973; LCSC Part C115056 -> C85973
- L1: value 1Kohm_100Mhz -> 220Ω@100MHz; LCSC Part C307758 -> C76815; MPN BLM15HG102SN1D -> MPZ1608S221ATA00
Connections:
- net FSM_button: now also C28.2
- net GND: now also C28.1, R5.1
- net at U1.60 (BOOT0): now also R5.2
- net ACEL_INT1 renamed INT2_ADXL
- net ACEL_INT2 renamed INT1_ADXL
- net DPS_INT renamed BMP_INT

Commit message: correcciones claude
Connections:
- net +3.3V: now also U1.1 (VBAT)
- no-connect marks 11 -> 10
Changed lines of the file:
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@@
-	)
-	(no_connect
-		(at 247.65 48.26)
 	)
 	(no_connect
@@
 		)
 		(stroke
+			(width 0)
+			(type default)
+		)
+	)
+	(wire
+		(pts
+			(xy 247.65 48.26) (xy 247.65 53.34)
+		)
+		(stroke

Commit message: 08/08
Connections:
- net WAKE_BNO: now reaches U1.57 (PB5)
- no-connect marks 10 -> 9
Changed lines of the file:
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@@
 	)
 	(no_connect
-		(at 302.26 146.05)
-	)
-	(no_connect
 		(at 302.26 179.07)
 	)
@@
 			)
 		)
+	)
+	(global_label "WAKE_BNO"
+		(shape input)
+		(at 302.26 146.05 0)
+		(fields_autoplaced yes)
+		(effects
+			(font
+				(size 1.27 1.27)
+			)
+			(justify left)
+		)
+		(property "Intersheetrefs" "${INTERSHEET_REFS}"
+			(at 315.1028 146.05 0)
+			(hide yes)
+			(show_name no)
+			(do_not_autoplace no)
+			(effects
+				(font
+					(size 1.27 1.27)
+				)
+				(justify left)
+			)
+		)
