File: POWER_V.kicad_sch (KiCad schematic)
At the start: 17 parts, among them CN1 XT30PW-M, CN2 XT30PW-M, SW1 SWITCH_BLACK, SW2 SWITCH_BLACK, U14 XL4005E1, U15 XC6220B331MR

Commit message: Arreglos de esquemático
Parts:
- added C9: 100nF, Capacitor_SMD:C_0402_1005Metric_Pad0.74x0.62mm_HandSolder, symbol CANSAT_STM32_symbols:TCC0402X7R104J500AT
- added LED1, LED2: (no value), Diode_SMD:D_0603_1608Metric_Pad1.05x0.95mm_HandSolder, symbol CANSAT_STM32_symbols:D-G060306G1-KS2
- added R14: 4.7K, easyeda2kicad:R0603, symbol CANSAT_STM32_symbols:RC0603FR-074K7L
- added R19: 10K, Resistor_SMD:R_0603_1608Metric_Pad0.98x0.95mm_HandSolder, symbol CANSAT_STM32_symbols:RC0603FR-7W10KL
- added TP4: TestPoint, TestPoint:TestPoint_Pad_D1.5mm, symbol Connector:TestPoint
- C40: footprint Capacitor_SMD:C_0603_1608Metric -> Capacitor_SMD:C_0603_1608Metric_Pad1.08x0.95mm_HandSolder
- R16, R17: footprint Capacitor_SMD:C_0603_1608Metric_Pad1.08x0.95mm_HandSolder -> Resistor_SMD:R_0603_1608Metric_Pad0.98x0.95mm_HandSolder
Connections:
- net +3V3: now also R14.2
- net +5V: now also R19.2
- net +BATT2: now also TP4.1
- net +VIN: now also C9.2
- net GND: now also C9.1, LED1.1 (-), LED2.1 (-)
- new net: LED2.2 (+), R19.1
- new net: LED1.2 (+), R14.1
Other:
- moved on the sheet: C38, C40, TP1, TP2, TP3, U15

Commit message: Arreglando footprints
Parts:
- removed C8: 220uF, ARLISS-footprints:CAP-TH_BD8.0-P3.50-D0.6-FD, symbol CANSAT_STM32_symbols:ECR1EBK221MLL080011
- added C32: 220uF, ARLISS-footprints:CAP-TH_BD8.0-P3.50-D0.6-FD, symbol Device:C_Polarized_US
- C31: renamed from C9; footprint Capacitor_SMD:C_0402_1005Metric_Pad0.74x0.62mm_HandSolder -> Capacitor_SMD:C_0603_1608Metric_Pad1.08x0.95mm_HandSolder; Manufacturer CCTC(三环) -> (none)
- C34: renamed from C10; Manufacturer Jianghai(南通江海) -> (none)
- LED4: renamed from LED2; Manufacturer ARKLED(方舟) -> (none)
- LED5: renamed from LED1; Manufacturer ARKLED(方舟) -> (none)
- R15: renamed from R19; Manufacturer YAGEO(国巨) -> (none)
- R16: renamed from R14; footprint easyeda2kicad:R0603 -> Resistor_SMD:R_0603_1608Metric_Pad0.98x0.95mm_HandSolder; Manufacturer YAGEO(国巨) -> (none)
- SW3: renamed from SW1; Manufacturer XKB Connection(中国星坤) -> (none)
- SW4: renamed from SW2; Manufacturer XKB Connection(中国星坤) -> (none)
- TP1: renamed from TP4; now left out of the parts list
- TP2: renamed from TP1; now left out of the parts list
- TP3: renamed from TP2; now left out of the parts list
- TP4: renamed from TP3; now left out of the parts list
- U7: renamed from U14; Manufacturer XLSEMI(芯龙) -> (none)
- renumbered C38 to C33, C40 to C35, D4 to D3, R16 to R13, R17 to R14, U15 to U8
Connections:
- net +VIN: now also C32.1
- net GND: now also C32.2
Other:
- company: (none) -> TOMEK TEAM

Commit message: Todo antes de PCB
Parts:
- removed C32: 220uF, ARLISS-footprints:CAP-TH_BD8.0-P3.50-D0.6-FD, symbol Device:C_Polarized_US
- removed C33: 10uF, Capacitor_SMD:C_0603_1608Metric_Pad1.08x0.95mm_HandSolder, symbol Device:C
- removed C34: 330uF, ARLISS-footprints:CAP-TH_BD10.0-P5.00-D1.0-FD, symbol CANSAT_STM32_symbols:ECR1EPT331MLL100012
- removed C35: 4.7uF, Capacitor_SMD:C_0603_1608Metric_Pad1.08x0.95mm_HandSolder, symbol Device:C
- removed D3: MBRD1060, Package_TO_SOT_SMD:TO-252-2, symbol Device:D_Schottky_AKA
- removed L2: 33uH, Inductor_SMD:L_APV_APH0850, symbol Device:L
- removed LED5: (no value), Diode_SMD:D_0603_1608Metric_Pad1.05x0.95mm_HandSolder, symbol CANSAT_STM32_symbols:D-G060306G1-KS2
- removed R15: 10K, Resistor_SMD:R_0603_1608Metric_Pad0.98x0.95mm_HandSolder, symbol CANSAT_STM32_symbols:RC0603FR-7W10KL
- removed U7: XL4005E1, ARLISS-footprints:TO-263-5_L10.2-W9.2-P1.70-TL, symbol CANSAT_STM32_symbols:XL4005E1
- removed U8: XC6220B331MR, Package_TO_SOT_SMD:SOT-23-5, symbol Regulator_Linear:XC6220B331MR
- added C32: 10uF, Capacitor_SMD:C_0805_2012Metric_Pad1.18x1.45mm_HandSolder, symbol CANSAT_STM32_symbols:TCC0402X7R104J500AT
- added C33: 4.7nF, Capacitor_SMD:C_0805_2012Metric_Pad1.18x1.45mm_HandSolder, symbol CANSAT_STM32_symbols:TCC0402X7R104J500AT
- added L2: 1uH, ARLISS-footprints:IND-SMD_L4.0-W4.0_XAL4030-332MEC, symbol CANSAT_STM32_symbols:XGL4020-102MEC
- added U7: TPS62901RPJR, ARLISS-footprints:VQFN-HR-9_L2.0-W1.5-P0.50-BL_TI_RPJ, symbol CANSAT_STM32_symbols:TPS62901RPJR
- C31: value 100nF -> 22uF; footprint Capacitor_SMD:C_0603_1608Metric_Pad1.08x0.95mm_HandSolder -> Capacitor_SMD:C_0805_2012Metric_Pad1.18x1.45mm_HandSolder; LCSC Part C5448844 -> C258782; MPN TCC0402X7R104J500AT -> GRM21BC81C226ME44L
- R13: value 12k -> 61.9k; LCSC C114659 -> C23091; Link https://www.lcsc.com/product-detail/C114659.html -> https://www.lcsc.com/datasheet/C23091.pdf?spm=wm.sxq.inf.gg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
- R14: value 2.2k -> 249k; LCSC C114662 -> C54531323; Link https://www.lcsc.com/product-detail/C114662.html -> https://www.lcsc.com/datasheet/C54531323.pdf?spm=wm.sxq.inf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
Connections:
- net FB is gone; now on net GND: R13.1, R14.2
- net +3V3: no longer R16.2
- net +BATT2: no longer TP1.1
- net +VIN: now also TP2.1, C32.2, U7.5 (EN), U7.6 (VIN); no longer C31.2
- net +VIN2: now also TP1.1
- net GND: now also C32.1, C33.2, U7.4 (GND); no longer R14.1
- net at LED4.2 (+): now also R16.1
- net +5V: no longer names the net of R13.2
- net +5V: now also U7.7 (MODE/S-CONF); no longer TP2.1
- new net: R14.1, U7.9 (FB/VSET)
- new net: L2.2, U7.2 (SW), U7.3 (VOS)
- new net: C33.1, U7.8 (SS/TR)
- new net +3.3V: C31.2, L2.1, R16.2
- no-connect marks 4 -> 5
Other:
- moved on the sheet: C31, LED4, R13, TP1, TP3, TP4
