File: POWER_V.kicad_sch (KiCad schematic)
At the start: 17 parts, among them CN1 XT30PW-M, CN2 XT30PW-M, SW3 SWITCH_BLACK, SW4 SWITCH_BLACK, U7 TPS62901RPJR

Commit message: Avance 02/08
Parts:
- C33: footprint Capacitor_SMD:C_0805_2012Metric_Pad1.18x1.45mm_HandSolder -> Capacitor_SMD:C_0603_1608Metric_Pad1.08x0.95mm_HandSolder
Other:
- note added: "CIN = C1"
- note added: "CSS/TR soft start"

Commit message: FINAL SCHEMATIC
Parts:
- R13: value 61.9k -> 76.8k; LCSC C23091 -> C165743; Link https://www.lcsc.com/datasheet/C23091.pdf?spm=wm.sxq.inf.gg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 -> https://www.lcsc.com/product-detail/C165743.html?spm=wm.fly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
Connections:
- net +3.3V: now also U7.3 (VOS)
- net at L2.2, U7.2 (SW): no longer U7.3 (VOS)
Other:
- note added: "R13 configuración"

Commit message: correcciones claude
Connections:
- net +VIN: no longer C32.2, U7.5 (EN), U7.6 (VIN)
- new net: C32.2, U7.5 (EN), U7.6 (VIN)
Changed lines of the file:
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@@
-	)
-	(symbol
-		(lib_id "power:+BATT")
-		(at 207.01 90.17 180)
-		(unit 1)
-		(body_style 1)
-		(exclude_from_sim no)
-		(in_bom yes)
-		(on_board yes)
-		(in_pos_files yes)
-		(dnp no)
-		(property "Reference" "#PWR084"
-			(at 207.01 86.36 0)
-			(hide yes)
-			(show_name no)
-			(do_not_autoplace no)
-			(effects
-				(font
-					(size 1.27 1.27)
-				)
-			)
-		)
-		(property "Value" "+VIN"
-			(at 209.296 94.742 0)
-			(show_name no)
-			(do_not_autoplace no)
-			(effects
-				(font
-					(size 1.27 1.27)
-				)
-				(justify left)
-			)
-		)
-		(property "Footprint" ""
-			(at 207.01 90.17 0)
-			(hide yes)
-			(show_name no)
-			(do_not_autoplace no)
-			(effects
-				(font
-					(size 1.27 1.27)
-				)
-			)
-		)
-		(property "Datasheet" ""
-			(at 207.01 90.17 0)
-			(hide yes)
-			(show_name no)
-			(do_not_autoplace no)
-			(effects
-				(font
-					(size 1.27 1.27)
-				)
-			)
-		)
-		(property "Description" "Power symbol creates a global label with name \"+BATT\""
-			(at 207.01 90.17 0)
-			(hide yes)
-			(show_name no)
-			(do_not_autoplace no)
-			(effects
-				(font
-					(size 1.27 1.27)
-				)
-			)
-		)
-		(pin "1"
-		)
-		(instances
-			(project "ARLISS_STM32_2026"
-				(path "/9719ea46-14c4-4409-9c57-49dd5454c03f/8549a18f-8dc0-4c64-a4df-732ef1c8a382"
-					(reference "#PWR084")
-					(unit 1)
-				)
-			)
-		)
 	)
 	(symbol
@@
 					(unit 1)
 				)
+			)
+		)
+	)
+	(symbol
+		(lib_name "+3V3_1")
+		(lib_id "power:+3V3")
+		(at 207.01 90.17 0)
+		(mirror x)
+		(unit 1)
+		(body_style 1)
+		(exclude_from_sim no)
+		(in_bom yes)
+		(on_board yes)
+		(in_pos_files yes)
+		(dnp no)
+		(fields_autoplaced yes)
+		(property "Reference" "#PWR0141"
+			(at 207.01 86.36 0)
+			(hide yes)
+			(show_name no)
+			(do_not_autoplace no)
+			(effects
+				(font
+					(size 1.27 1.27)
+				)
+			)
+		)
+		(property "Value" "VINS+"
+			(at 207.01 95.25 0)
+			(show_name no)
+			(do_not_autoplace no)
+			(effects
+				(font
+					(size 1.27 1.27)
+				)
+			)
+		)
+		(property "Footprint" ""
+			(at 207.01 90.17 0)
+			(hide yes)
+			(show_name no)
+			(do_not_autoplace no)
+			(effects
+				(font
+					(size 1.27 1.27)
+				)
+			)
+		)
+		(property "Datasheet" ""
+			(at 207.01 90.17 0)
+			(hide yes)
+			(show_name no)
+			(do_not_autoplace no)
+			(effects
+				(font
+					(size 1.27 1.27)
+				)
+			)
+		)
+		(property "Description" "Power symbol creates a global label with name \"+3V3\""
+			(at 207.01 90.17 0)
+			(hide yes)
+			(show_name no)
+			(do_not_autoplace no)
+			(effects
+				(font
+					(size 1.27 1.27)
+				)
+			)
+		)
+		(pin "1"
+		)
+		(instances
+			(project "ARLISS_STM32_2026"
+				(path "/9719ea46-14c4-4409-9c57-49dd5454c03f/8549a18f-8dc0-4c64-a4df-732ef1c8a382"
+					(reference "#PWR0141")
+					(unit 1)
+				)

Commit message: 08/08
Parts:
- added D3, D4: D_Zener, Diode_SMD:D_SOD-123, symbol Device:D_Zener
- added F1: 7A, ARLISS-footprints:F1206, symbol CANSAT_STM32_symbols:LTC1206-1700TS
- added F2: 750mA, ARLISS-footprints:F1206, symbol CANSAT_STM32_symbols:0466.750NRHF
- added LED6: (no value), Diode_SMD:D_0603_1608Metric_Pad1.05x0.95mm_HandSolder, symbol CANSAT_STM32_symbols:D-G060306G1-KS2
- added Q2, Q3: AOD4185_C400894, ARLISS-footprints:TO-252-3_L6.6-W6.1-P4.57-LS9.9-BR-CW, symbol CANSAT_STM32_symbols:AOD4185_C400894
- added R27, R28: 100k, Resistor_SMD:R_0603_1608Metric_Pad0.98x0.95mm_HandSolder, symbol CANSAT_STM32_symbols:RC0603FR-07100KL
- added R29, R30: TLRZ2ATTD, ARLISS-footprints:R0805, symbol CANSAT_STM32_symbols:TLRZ2ATTD
- added RIPROPI3: 2.4K, Resistor_SMD:R_0603_1608Metric_Pad0.98x0.95mm_HandSolder, symbol Device:R
Connections:
- net +3.3V: now also RIPROPI3.1; no longer R16.2
- net +VIN: now also F2.2, R30.1
- net +VIN2: now also F1.2, R29.1
- net GND: now also LED6.1 (-), R27.1, R28.1
- net at LED4.2 (+): now also RIPROPI3.2; no longer R16.1
- new net: D3.2 (A), Q2.1 (G), R27.2
- new net: F1.1, Q2.2 (D)
- new net: F2.1, Q3.2 (D)
- new net: D4.2 (A), Q3.1 (G), R28.2
- new net: LED6.2 (+), R16.1
- new net +11.1V: R16.2
- new net +VIN2P: D3.1 (K), Q2.3 (S), R29.2
- new net +VINP: D4.1 (K), Q3.3 (S), R30.2
Other:
- moved on the sheet: C31, C32, C33, L2, LED4, R13, R14, U7
