File: POWER_V.kicad_sch (KiCad schematic)
At the start: 29 parts, among them CN1 XT30PW-M, CN2 XT30PW-M, Q2 AOD4185_C400894, Q3 AOD4185_C400894, SW3 SWITCH_BLACK, SW4 SWITCH_BLACK, U7 TPS62901RPJR

Commit message: SCHEMATICO TOTAL
Parts:
- C31: LCSC Part C258782 -> C342717; MPN GRM21BC81C226ME44L -> C2012X7S1A226MT000E
- renumbered RIPROPI3 to R4
Connections:
- net +3V3 is gone; now on net +3.3V: TP4.1
- net +11.1V: now also TP1.1
- net +VIN2: no longer TP1.1
Other:
- moved on the sheet: TP1, TP2, TP3, TP4

Commit message: PCB_V1
Parts:
- added D1: SMBJ10A_C151250, ARLISS-footprints:SMB_L4.6-W3.6-LS5.3-RD, symbol CANSAT_STM32_symbols:SMBJ10A_C151250
- added TP5: TestPoint, TestPoint:TestPoint_Pad_D1.5mm, symbol Connector:TestPoint
Connections:
- net +VIN2: now also TP5.1
- net +VINP: now also D1.1 (K)
- net GND: now also D1.2 (A)
Other:
- moved on the sheet: D3, F1, Q2, R27, TP3, TP4

Commit message: Cambios finales antes de main
Parts:
- added JP1, JP2, JP3, JP4: SolderJumper_2_Open, Jumper:SolderJumper-2_P1.3mm_Open_TrianglePad1.0x1.5mm, symbol Jumper:SolderJumper_2_Open
- added LED7, LED8: (no value), Diode_SMD:D_0603_1608Metric_Pad1.05x0.95mm_HandSolder, symbol CANSAT_STM32_symbols:D-G060306G1-KS2
- added R32: 2.4K, Resistor_SMD:R_0603_1608Metric_Pad0.98x0.95mm_HandSolder, symbol Device:R
- added R33: 4.7K, Resistor_SMD:R_0603_1608Metric_Pad0.98x0.95mm_HandSolder, symbol CANSAT_STM32_symbols:RC0603FR-074K7L
Connections:
- net +VIN: now also R32.1
- net +VIN2: now also R33.2
- net GND: now also JP1.2 (B), JP2.2 (B), JP3.2 (B), JP4.2 (B); no longer LED4.1 (-), LED6.1 (-)
- new net: JP1.1 (A), LED4.1 (-)
- new net: JP3.1 (A), LED7.1 (-)
- new net: JP2.1 (A), LED6.1 (-)
- new net: JP4.1 (A), LED8.1 (-)
- new net: LED8.2 (+), R32.2
- new net: LED7.2 (+), R33.1

Commit message: PCB_2.0
Parts:
- removed JP2: SolderJumper_2_Open, Jumper:SolderJumper-2_P1.3mm_Open_TrianglePad1.0x1.5mm, symbol Jumper:SolderJumper_2_Open
- removed LED6: (no value), Diode_SMD:D_0603_1608Metric_Pad1.05x0.95mm_HandSolder, symbol CANSAT_STM32_symbols:D-G060306G1-KS2
- removed R16, R33: 4.7K, Resistor_SMD:R_0603_1608Metric_Pad0.98x0.95mm_HandSolder, symbol CANSAT_STM32_symbols:RC0603FR-074K7L
- removed R32: 2.4K, Resistor_SMD:R_0603_1608Metric_Pad0.98x0.95mm_HandSolder, symbol Device:R
- added R16: 10K, Resistor_SMD:R_0603_1608Metric_Pad0.98x0.95mm_HandSolder, symbol CANSAT_STM32_symbols:RC0603FR-7W10KL
- added R34: 4.7K, Resistor_SMD:R_0603_1608Metric_Pad0.98x0.95mm_HandSolder, symbol CANSAT_STM32_symbols:RC0603FR-074K7L
- added TP6: TestPoint, TestPoint:TestPoint_Pad_D1.5mm, symbol Connector:TestPoint
Connections:
- net +3.3V: now also JP1.1 (A); no longer R4.1
- net +VIN: now also JP4.1 (A)
- net +VIN2: now also JP3.1 (A)
- net GND: now also LED4.1 (-), LED7.1 (-), LED8.1 (-), TP6.1; no longer JP1.2 (B), JP3.2 (B), JP4.2 (B)
- net at LED8.2 (+): now also R34.1
- net at LED7.2 (+): now also R16.1
- new net: JP3.2 (B), R16.2
- new net: JP4.2 (B), R34.2
- new net: JP1.2 (B), R4.1
Other:
- moved on the sheet: JP1, JP3, LED4, LED7, LED8, R4

Commit message: jhamir
Other:
- moved on the sheet: CN2, D1, D3, F1, JP1, JP3, LED4, LED7, Q2, R27, R29, R30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

Commit message: ordenando
Parts:
- removed JP1, JP3, JP4: SolderJumper_2_Open, Jumper:SolderJumper-2_P1.3mm_Open_TrianglePad1.0x1.5mm, symbol Jumper:SolderJumper_2_Open
Connections:
- net +3.3V: now also R4.1
- net +VIN: now also R34.2
- net +VIN2: now also R16.2
Other:
- moved on the sheet: LED4, LED7, LED8, R16, R34, R4
