File: DriverDRV8874.kicad_sch (KiCad schematic)
At the start: 26 parts, among them J1 Conn_01x06, J2 Conn_01x06, U3 DRV8874PWPR, U4 DRV8874PWPR

Commit message: 08/08
Connections:
- net +VINS2 is gone; now on net +11.1V: U3.11 (VM), U4.11 (VM)
- net +VIN2 renamed +11.1V

Commit message: SCHEMATICO TOTAL
Parts:
- removed D1, D2: SMBJ18A_C151256, ARLISS-footprints:SMB_L4.3-W3.6-LS5.3-RD, symbol CANSAT_STM32_symbols:SMBJ18A_C151256
- removed R10, R9: 1K, Resistor_SMD:R_0603_1608Metric_Pad0.98x0.95mm_HandSolder, symbol CANSAT_STM32_symbols:RC0603FR-071KL
- added D5, D6: SMBJ18CA_C83327, easyeda2kicad:SMB_L4.6-W3.6-LS5.3-BI, symbol CANSAT_STM32_symbols:SMBJ18CA_C83327
- added R10, R9: 2.4K, Resistor_SMD:R_0603_1608Metric_Pad0.98x0.95mm_HandSolder, symbol Device:R
Connections:
- net +11.1V: now also D5.1 (K), D6.1 (K)
- net GND: now also D5.2 (A), D6.2 (A)
- net at LED2.2 (+): now also R9.2
- net at LED3.2 (+): now also R10.2
- net +3V3 renamed +3.3V
- net +3.3V: now also R10.1, R9.1

Commit message: PCB_V1
Parts:
- D5, D6: footprint easyeda2kicad:SMB_L4.6-W3.6-LS5.3-BI -> ARLISS-footprints:SMB_L4.6-W3.6-LS5.3-BI
Changed lines of the file:
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@@
 			)
 		)
-		(property "Footprint" "easyeda2kicad:SMB_L4.6-W3.6-LS5.3-BI"
+		(property "Footprint" "ARLISS-footprints:SMB_L4.6-W3.6-LS5.3-BI"
 			(at 217.17 72.39 0)
 			(hide yes)
@@
 			)
 		)
-		(property "Footprint" "easyeda2kicad:SMB_L4.6-W3.6-LS5.3-BI"
+		(property "Footprint" "ARLISS-footprints:SMB_L4.6-W3.6-LS5.3-BI"
 			(at 214.63 143.51 0)
 			(hide yes)

Commit message: PCB_2.0
Parts:
- renumbered RIMODE1 to RIM1, RIMODE2 to RIM2, RIPROPI1 to RIPR1, RIPROPI2 to RIPR2
Changed lines of the file:
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@@
 		(dnp no)
 		(fields_autoplaced yes)
-		(property "Reference" "RIMODE2"
+		(property "Reference" "RIM2"
 			(at 265.43 38.0999 0)
 			(show_name no)
@@
 			(project "ARLISS_STM32_2026"
 				(path "/9719ea46-14c4-4409-9c57-49dd5454c03f/4b4c1a4f-7753-466f-b706-7dda6e0dceb5"
-					(reference "RIMODE2")
+					(reference "RIM2")
 					(unit 1)
 				)
@@
 		(in_pos_files yes)
 		(dnp no)
-		(property "Reference" "RIPROPI2"
+		(property "Reference" "RIPR2"
 			(at 138.938 128.524 0)
 			(show_name no)
@@
 			(project "ARLISS_STM32_2026"
 				(path "/9719ea46-14c4-4409-9c57-49dd5454c03f/4b4c1a4f-7753-466f-b706-7dda6e0dceb5"
-					(reference "RIPROPI2")
+					(reference "RIPR2")
 					(unit 1)
 				)
@@
 		(in_pos_files yes)
 		(dnp no)
-		(property "Reference" "RIPROPI1"
+		(property "Reference" "RIPR1"
 			(at 138.938 62.484 0)
 			(show_name no)
@@
 			(project "ARLISS_STM32_2026"
 				(path "/9719ea46-14c4-4409-9c57-49dd5454c03f/4b4c1a4f-7753-466f-b706-7dda6e0dceb5"
-					(reference "RIPROPI1")
+					(reference "RIPR1")
 					(unit 1)
 				)
@@
 		(dnp no)
 		(fields_autoplaced yes)
-		(property "Reference" "RIMODE1"
+		(property "Reference" "RIM1"
 			(at 260.35 106.6799 0)
 			(show_name no)
@@
 			(project "ARLISS_STM32_2026"
 				(path "/9719ea46-14c4-4409-9c57-49dd5454c03f/4b4c1a4f-7753-466f-b706-7dda6e0dceb5"
-					(reference "RIMODE1")
-					(unit 1)
-				)
+					(reference "RIM1")
+					(unit 1)
+				)

Commit message: ordenando
Parts:
- removed D5, D6: SMBJ18CA_C83327, ARLISS-footprints:SMB_L4.6-W3.6-LS5.3-BI, symbol CANSAT_STM32_symbols:SMBJ18CA_C83327
- added C31, C32: 10uF, Capacitor_SMD:C_0805_2012Metric_Pad1.18x1.45mm_HandSolder, symbol CANSAT_STM32_symbols:CL21B106KAYQNNE
- R10, R9, RIPR1, RIPR2: value 2.4K -> 2.2K; LCSC C114611 -> C125931
Connections:
- net +11.1V: now also C31.2, C32.2
- net GND: now also C31.1, C32.1
Other:
- moved on the sheet: C15, C18, C20, C21, C23, C24, C25, LED2, RIM1, RIPR2, U4

Commit message: FINAL
Parts:
- J1: LCSC (none) -> C144397; LINK (none) -> https://www.lcsc.com/datasheet/C144397.pdf?spm=wm.sxq.inf.g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
Changed lines of the file:
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@@
 			)
 		)
-		(property "Field7" ""
+		(property "LCSC" "C144397"
 			(at 124.46 173.99 0)
 			(hide yes)
+			(show_name no)
+			(do_not_autoplace no)
+			(effects
+				(font
+					(size 1.27 1.27)
+				)
+			)
+		)
+		(property "LINK" "https://www.lcsc.com/datasheet/C144397.pdf?spm=wm.sxq.inf.ggs___wm.ssy.bg.10.xh&lcsc_vid=T1RYXlBeQ1NXVVRQElQIBgFfEVVfUlADQlYNVlEFRFIxVlNeQFNaUFBRRFZeVzsOAxUeFF5JWBYZEEoKFBINSQcJGk4%3D"
+			(at 124.46 173.99 0)
+			(hide yes)
