File: Barómetro Botch SMD.kicad_sch (KiCad schematic)
At the start: 3 parts, among them U5 BMP581

Commit message: FINAL SCHEMATIC
Changed lines of the file:
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@@
 	(wire
 		(pts
-			(xy 132.08 72.39) (xy 134.62 72.39)
+			(xy 132.08 72.39) (xy 143.51 72.39)
 		)
 		(stroke
@@
 		)
 	)
+	(label "VDDIO"
+		(at 95.25 62.23 0)
+		(effects
+			(font
+				(size 1.27 1.27)
+			)
+			(justify left bottom)
+		)
+	)
+	(label "VDDIO"
+		(at 143.51 72.39 0)
+		(effects
+			(font
+				(size 1.27 1.27)
+			)
+			(justify left bottom)
+		)
+	)
 	(global_label "I2C1_SDA"
 		(shape input)
@@
 			)
 		)
-	)
-	(symbol
-		(lib_id "power:+3.3V")
-		(at 134.62 72.39 180)
-		(unit 1)
-		(body_style 1)
-		(exclude_from_sim no)
-		(in_bom yes)
-		(on_board yes)
-		(in_pos_files yes)
-		(dnp no)
-		(fields_autoplaced yes)
-		(property "Reference" "#PWR068"
-			(at 134.62 68.58 0)
-			(hide yes)
-			(show_name no)
-			(do_not_autoplace no)
-			(effects
-				(font
-					(size 1.27 1.27)
-				)
-			)
-		)
-		(property "Value" "+3.3V"
-			(at 134.62 77.47 0)
-			(show_name no)
-			(do_not_autoplace no)
-			(effects
-				(font
-					(size 1.27 1.27)
-				)
-			)
-		)
-		(property "Footprint" ""
-			(at 134.62 72.39 0)
-			(hide yes)
-			(show_name no)
-			(do_not_autoplace no)
-			(effects
-				(font
-					(size 1.27 1.27)
-				)
-			)
-		)
-		(property "Datasheet" ""
-			(at 134.62 72.39 0)
-			(hide yes)
-			(show_name no)
-			(do_not_autoplace no)
-			(effects
-				(font
-					(size 1.27 1.27)
-				)
-			)
-		)
-		(property "Description" "Power symbol creates a global label with name \"+3.3V\""
-			(at 134.62 72.39 0)
-			(hide yes)
-			(show_name no)
-			(do_not_autoplace no)
-			(effects
-				(font
-					(size 1.27 1.27)
-				)
-			)
-		)
-		(pin "1"
-		)
-		(instances
-			(project "ARLISS_STM32_2026"
-				(path "/9719ea46-14c4-4409-9c57-49dd5454c03f/9e299f07-4887-409a-8623-587b30453872"
-					(reference "#PWR068")
-					(unit 1)
-				)
-			)
-		)

Commit message: SCHEMATICO TOTAL
Changed lines of the file:
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@@
 	)
 	(junction
+		(at 95.25 62.23)
+		(diameter 0)
+		(color 0 0 0 0)
+	)
+	(junction
 		(at 132.08 67.31)
 		(diameter 0)
@@
 	(wire
 		(pts
-			(xy 132.08 72.39) (xy 143.51 72.39)
+			(xy 95.25 60.96) (xy 95.25 62.23)
+		)
+		(stroke
+			(width 0)
+			(type default)
+		)
+	)
+	(wire
+		(pts
+			(xy 142.24 72.39) (xy 132.08 72.39)
+		)
+		(stroke
+			(width 0)
+			(type default)
+		)
+	)
+	(wire
+		(pts
+			(xy 142.24 83.82) (xy 142.24 72.39)
+		)
+		(stroke
+			(width 0)
+			(type default)
+		)
+	)
+	(wire
+		(pts
+			(xy 142.24 83.82) (xy 146.05 83.82)
 		)
 		(stroke
@@
 	(wire
 		(pts
-			(xy 82.55 62.23) (xy 109.22 62.23)
+			(xy 82.55 62.23) (xy 95.25 62.23)
+		)
+		(stroke
+			(width 0)
+			(type default)
+		)
+	)
+	(wire
+		(pts
+			(xy 95.25 62.23) (xy 109.22 62.23)
 		)
 		(stroke
@@
 	)
 	(label "VDDIO"
-		(at 95.25 62.23 0)
+		(at 95.25 60.96 0)
 		(effects
 			(font
@@
 	)
 	(label "VDDIO"
-		(at 143.51 72.39 0)
+		(at 146.05 83.82 0)
 		(effects
 			(font
