File: NICROM.kicad_sch (KiCad schematic)
At the start: 5 parts, among them J3 Screw_Terminal_01x02, Q1 IRLZ44NPBF

Commit message: Avance 02/08
Parts:
- added LED5: D-R060306L3-KS2, Diode_SMD:D_0603_1608Metric_Pad1.05x0.95mm_HandSolder, symbol CANSAT_STM32_symbols:D-R060306L3-KS2
Connections:
- net GND: now also LED5.1 (-)
- net Led_Mosfet: now also LED5.2 (+)
Changed lines of the file:
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@@
+	)
+	(symbol
+		(lib_id "CANSAT_STM32_symbols:D-R060306L3-KS2")
+		(at 88.9 113.03 90)
+		(unit 1)
+		(body_style 1)
+		(exclude_from_sim no)
+		(in_bom yes)
+		(on_board yes)
+		(in_pos_files yes)
+		(dnp no)
+		(fields_autoplaced yes)
+		(property "Reference" "LED5"
+			(at 93.98 114.2999 90)
+			(show_name no)
+			(do_not_autoplace no)
+			(effects
+				(font
+					(size 1.27 1.27)
+				)
+				(justify right)
+			)
+		)
+		(property "Value" "D-R060306L3-KS2"
+			(at 93.98 114.3 0)
+			(hide yes)
+			(show_name no)
+			(do_not_autoplace no)
+			(effects
+				(font
+					(size 1.27 1.27)
+				)
+			)
+		)
+		(property "Footprint" "Diode_SMD:D_0603_1608Metric_Pad1.05x0.95mm_HandSolder"
+			(at 97.79 113.03 0)
+			(hide yes)
+			(show_name no)
+			(do_not_autoplace no)
+			(effects
+				(font
+					(size 1.27 1.27)
+				)
+			)
+		)
+		(property "Datasheet" "https://lcsc.com/product-detail/Light-Emitting-Diodes-LED_D-R060306L3-KS2-Azarin_C118330.html"
+			(at 100.33 113.03 0)
+			(hide yes)
+			(show_name no)
+			(do_not_autoplace no)
+			(effects
+				(font
+					(size 1.27 1.27)
+				)
+			)
+		)
+		(property "Description" ""
+			(at 88.9 113.03 0)
+			(hide yes)
+			(show_name yes)
+			(do_not_autoplace no)
+			(effects
+				(font
+					(size 1.27 1.27)
+				)
+			)
+		)
+		(property "MPN" "D-060306R1/SS2/L"
+			(at 105.41 113.03 0)
+			(hide yes)
+			(show_name no)
+			(do_not_autoplace no)
+			(effects
+				(font
+					(size 1.27 1.27)
+				)
+			)
+		)
+		(property "LCSC Part" "C118330"
+			(at 107.95 113.03 0)
+			(hide yes)
+			(show_name no)
+			(do_not_autoplace no)
+			(effects
+				(font
+					(size 1.27 1.27)
+				)
+			)
+		)
+		(property "Field7" ""
+			(at 88.9 113.03 0)
+			(hide yes)
+			(show_name no)
+			(do_not_autoplace no)
+			(effects
+				(font
+					(size 1.27 1.27)
+				)
+			)
+		)
+		(pin "1"
+		)
+		(pin "2"
+		)
+		(instances
+			(project "ARLISS_STM32_2026"
+				(path "/9719ea46-14c4-4409-9c57-49dd5454c03f/5b57be68-8372-451f-98b5-1e3ec0294f41"
+					(reference "LED5")
+					(unit 1)
+				)
+			)
+		)
 	)
 	(symbol

Commit message: FINAL SCHEMATIC
Parts:
- R17, R18: footprint Capacitor_SMD:C_0603_1608Metric_Pad1.08x0.95mm_HandSolder -> Resistor_SMD:R_0603_1608Metric_Pad0.98x0.95mm_HandSolder
Connections:
- net Led_Mosfet: no longer names the net of LED5.2 (+), R17.1
Changed lines of the file:
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@@
-	)
-	(junction
-		(at 90.17 105.41)
-		(diameter 0)
-		(color 0 0 0 0)
 	)
 	(junction
@@
 	(wire
 		(pts
-			(xy 90.17 107.95) (xy 90.17 105.41)
+			(xy 123.19 86.36) (xy 123.19 90.17)
 		)
 		(stroke
@@
 	(wire
 		(pts
-			(xy 123.19 86.36) (xy 123.19 90.17)
+			(xy 129.54 121.92) (xy 129.54 125.73)
 		)
 		(stroke
@@
 	(wire
 		(pts
-			(xy 129.54 121.92) (xy 129.54 125.73)
+			(xy 138.43 104.14) (xy 138.43 121.92)
 		)
 		(stroke
@@
 	(wire
 		(pts
-			(xy 138.43 104.14) (xy 138.43 121.92)
+			(xy 123.19 99.06) (xy 130.81 99.06)
 		)
 		(stroke
@@
 	(wire
 		(pts
-			(xy 123.19 99.06) (xy 130.81 99.06)
+			(xy 138.43 76.2) (xy 138.43 80.01)
 		)
 		(stroke
@@
 	(wire
 		(pts
-			(xy 138.43 76.2) (xy 138.43 80.01)
+			(xy 88.9 93.98) (xy 90.17 93.98)
 		)
 		(stroke
@@
 	(wire
 		(pts
-			(xy 88.9 93.98) (xy 90.17 93.98)
+			(xy 123.19 115.57) (xy 123.19 121.92)
 		)
 		(stroke
@@
 	(wire
 		(pts
-			(xy 123.19 115.57) (xy 123.19 121.92)
-		)
-		(stroke
-			(width 0)
-			(type default)
-		)
-	)
-	(wire
-		(pts
-			(xy 83.82 105.41) (xy 90.17 105.41)
-		)
-		(stroke
-			(width 0)
-			(type default)
-		)
-	)
-	(wire
-		(pts
-			(xy 90.17 105.41) (xy 90.17 101.6)
+			(xy 90.17 101.6) (xy 90.17 107.95)
 		)
 		(stroke
@@
 		)
 	)
-	(label "Led_Mosfet"
-		(at 83.82 105.41 180)
-		(effects
-			(font
-				(size 1.27 1.27)
-			)
-			(justify right bottom)
-		)
-	)
 	(label "Mosfet_S"
 		(at 138.43 91.44 0)
@@
 			)
 		)
-		(property "Footprint" "Capacitor_SMD:C_0603_1608Metric_Pad1.08x0.95mm_HandSolder"
+		(property "Footprint" "Resistor_SMD:R_0603_1608Metric_Pad0.98x0.95mm_HandSolder"
 			(at 90.17 99.06 0)
 			(hide yes)
@@
 			)
 		)
-		(property "Footprint" "Capacitor_SMD:C_0603_1608Metric_Pad1.08x0.95mm_HandSolder"
+		(property "Footprint" "Resistor_SMD:R_0603_1608Metric_Pad0.98x0.95mm_HandSolder"
 			(at 123.19 92.71 0)
 			(hide yes)

Commit message: SCHEMATICO TOTAL
Parts:
- removed R17: 1k, Resistor_SMD:R_0603_1608Metric_Pad0.98x0.95mm_HandSolder, symbol Device:R_Small
- added R17: 2.4K, Resistor_SMD:R_0603_1608Metric_Pad0.98x0.95mm_HandSolder, symbol Device:R
Connections:
- net PIN_MOSFET: now also R17.1
- net at LED5.2 (+): now also R17.2
- net +VIN2 renamed +11.1V

Commit message: PCB_V1
Parts:
- Q1: footprint ARLISS-footprints:TO-220-3_L10.0-W4.5-P2.54-T -> Package_TO_SOT_THT:TO-220-3_Horizontal_TabDown
Changed lines of the file:
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@@
+		)
+	)
+	(text_box "Cambio probable a C878812\nR 100k->1M "
+		(exclude_from_sim no)
+		(at 55.88 59.69 0)
+		(size 36.83 12.7)
+		(margins 0.9525 0.9525 0.9525 0.9525)
+		(stroke
+			(width 0)
+			(type solid)
+		)
+		(fill
+			(type none)
+		)
+		(effects
+			(font
+				(size 1.27 1.27)
+			)
+			(justify left top)
 		)
 	)
@@
 			)
 		)
-		(property "Footprint" "ARLISS-footprints:TO-220-3_L10.0-W4.5-P2.54-T"
+		(property "Footprint" "Package_TO_SOT_THT:TO-220-3_Horizontal_TabDown"
 			(at 135.89 111.76 0)
 			(hide yes)

Commit message: ordenando
Parts:
- R17: value 2.4K -> 2.2K
Changed lines of the file:
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@@
 			)
 		)
-		(property "Value" "2.4K"
+		(property "Value" "2.2K"
 			(at 91.694 102.616 0)
 			(show_name no)

Commit message: 3D MODEL
Parts:
- removed J3: Screw_Terminal_01x02, TerminalBlock_RND:TerminalBlock_RND_205-00232_1x02_P5.08mm_Horizontal, symbol Connector:Screw_Terminal_01x02
- added CN3: DB127V-5.08-2P-GN-S, ARLISS-footprints:CONN-TH_2P-P5.08, symbol CANSAT_STM32_symbols:DB127V-5.08-2P-GN-S
Connections:
- net +11.1V: now also CN3.1
- net Mosfet_S: now also CN3.2
Changed lines of the file:
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@@
-	)
-	(symbol
-		(lib_id "Connector:Screw_Terminal_01x02")
-		(at 143.51 80.01 0)
-		(unit 1)
-		(body_style 1)
-		(exclude_from_sim no)
-		(in_bom yes)
-		(on_board yes)
-		(in_pos_files yes)
-		(dnp no)
-		(fields_autoplaced yes)
-		(property "Reference" "J3"
-			(at 146.05 80.0099 0)
-			(show_name no)
-			(do_not_autoplace no)
-			(effects
-				(font
-					(size 1.27 1.27)
-				)
-				(justify left)
-			)
-		)
-		(property "Value" "Screw_Terminal_01x02"
-			(at 146.05 82.5499 0)
-			(show_name no)
-			(do_not_autoplace no)
-			(effects
-				(font
-					(size 1.27 1.27)
-				)
-				(justify left)
-			)
-		)
-		(property "Footprint" "TerminalBlock_RND:TerminalBlock_RND_205-00232_1x02_P5.08mm_Horizontal"
-			(at 143.51 80.01 0)
-			(hide yes)
-			(show_name no)
-			(do_not_autoplace no)
-			(effects
-				(font
-					(size 1.27 1.27)
-				)
-			)
-		)
-		(property "Datasheet" ""
-			(at 143.51 80.01 0)
-			(hide yes)
-			(show_name no)
-			(do_not_autoplace no)
-			(effects
-				(font
-					(size 1.27 1.27)
-				)
-			)
-		)
-		(property "Description" "Generic screw terminal, single row, 01x02, script generated (kicad-library-utils/schlib/autogen/connector/)"
-			(at 143.51 80.01 0)
-			(hide yes)
-			(show_name no)
-			(do_not_autoplace no)
-			(effects
-				(font
-					(size 1.27 1.27)
-				)
-			)
-		)
-		(property "Link" "https://www.lcsc.com/product-detail/C8465.html?s_z=n_C8465"
-			(at 143.51 80.01 0)
-			(hide yes)
-			(show_name no)
-			(do_not_autoplace no)
-			(effects
-				(font
-					(size 1.27 1.27)
-				)
-			)
-		)
-		(property "Field7" ""
-			(at 143.51 80.01 0)
-			(hide yes)
-			(show_name no)
-			(do_not_autoplace no)
-			(effects
-				(font
-					(size 1.27 1.27)
-				)
-			)
-		)
-		(pin "2"
-		)
-		(pin "1"
-		)
-		(instances
-			(project "ARLISS_STM32_2026"
-				(path "/9719ea46-14c4-4409-9c57-49dd5454c03f/5b57be68-8372-451f-98b5-1e3ec0294f41"
-					(reference "J3")
-					(unit 1)
-				)
-			)
-		)
 	)
 	(symbol
@@
 					(unit 1)
 				)
+			)
+		)
+	)
+	(symbol
+		(lib_id "CANSAT_STM32_symbols:DB127V-5.08-2P-GN-S")
+		(at 142.24 81.28 0)
+		(unit 1)
+		(body_style 1)
+		(exclude_from_sim no)
+		(in_bom yes)
+		(on_board yes)
+		(in_pos_files yes)
+		(dnp no)
+		(fields_autoplaced yes)
+		(property "Reference" "CN3"
+			(at 147.32 80.0099 0)
+			(show_name no)
+			(do_not_autoplace no)
+			(effects
+				(font
+					(size 1.27 1.27)
+				)
+				(justify left)
+			)
+		)
+		(property "Value" "DB127V-5.08-2P-GN-S"
+			(at 147.32 82.5499 0)
+			(show_name no)
+			(do_not_autoplace no)
+			(effects
+				(font
+					(size 1.27 1.27)
+				)
+				(justify left)
+			)
+		)
+		(property "Footprint" "ARLISS-footprints:CONN-TH_2P-P5.08"
+			(at 142.24 90.17 0)
+			(hide yes)
+			(show_name no)
+			(do_not_autoplace no)
+			(effects
+				(font
+					(size 1.27 1.27)
+				)
+			)
+		)
+		(property "Datasheet" "https://www.lcsc.com/datasheet/C3018698.pdf"
+			(at 142.24 92.71 0)
+			(hide yes)
+			(show_name no)
+			(do_not_autoplace no)
+			(effects
+				(font
+					(size 1.27 1.27)
+				)
+			)
+		)
+		(property "Description" ""
+			(at 142.24 81.28 0)
+			(hide yes)
+			(show_name no)
+			(do_not_autoplace no)
+			(effects
+				(font
+					(size 1.27 1.27)
+				)
+			)
+		)
+		(property "Manufacturer" "DORABO(地博电气)"
+			(at 142.24 95.25 0)
+			(hide yes)
+			(show_name no)
+			(do_not_autoplace no)
+			(effects
+				(font
+					(size 1.27 1.27)
+				)
+			)
+		)
+		(property "MPN" "DB127V-5.08-2P-GN-S"
+			(at 142.24 97.79 0)
+			(hide yes)
+			(show_name no)
+			(do_not_autoplace no)
+			(effects
+				(font
+					(size 1.27 1.27)
+				)
+			)
+		)
+		(property "LCSC Part" "C3018698"
+			(at 142.24 100.33 0)
+			(hide yes)
+			(show_name no)
+			(do_not_autoplace no)
+			(effects
+				(font
+					(size 1.27 1.27)
+				)
+			)
+		)
+		(pin "1"
+		)
+		(pin "2"
+		)
+		(instances
+			(project "ARLISS_STM32_2026"
+				(path "/9719ea46-14c4-4409-9c57-49dd5454c03f/5b57be68-8372-451f-98b5-1e3ec0294f41"
+					(reference "CN3")
+					(unit 1)
+				)

Commit message: PLACA FINISHED
Parts:
- Q1: footprint Package_TO_SOT_THT:TO-220-3_Horizontal_TabDown -> Package_TO_SOT_THT:TO-220-3_Horizontal_TabUp
- R18: Link https://www.lcsc.com/product-detail/C859110.html -> (none)
Connections:
- net Mosfet_S renamed Mosfet_D
Changed lines of the file:
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@@
+	)
+	(junction
+		(at 138.43 111.76)
+		(diameter 0)
+		(color 0 0 0 0)
+	)
+	(junction
+		(at 138.43 91.44)
+		(diameter 0)
+		(color 0 0 0 0)
 	)
 	(junction
@@
 	)
 	(junction
-		(at 138.43 91.44)
-		(diameter 0)
-		(color 0 0 0 0)
-	)
-	(junction
 		(at 123.19 99.06)
 		(diameter 0)
@@
 	(wire
 		(pts
-			(xy 138.43 91.44) (xy 138.43 93.98)
+			(xy 143.51 111.76) (xy 138.43 111.76)
 		)
 		(stroke
@@
 	(wire
 		(pts
-			(xy 123.19 86.36) (xy 123.19 90.17)
+			(xy 138.43 91.44) (xy 142.24 91.44)
 		)
 		(stroke
@@
 	(wire
 		(pts
-			(xy 90.17 104.14) (xy 90.17 107.95)
+			(xy 123.19 86.36) (xy 123.19 90.17)
 		)
 		(stroke
@@
 	(wire
 		(pts
-			(xy 129.54 121.92) (xy 129.54 125.73)
+			(xy 90.17 104.14) (xy 90.17 107.95)
 		)
 		(stroke
@@
 	(wire
 		(pts
-			(xy 138.43 104.14) (xy 138.43 121.92)
+			(xy 129.54 121.92) (xy 129.54 125.73)
 		)
 		(stroke
@@
 	(wire
 		(pts
-			(xy 123.19 99.06) (xy 130.81 99.06)
+			(xy 138.43 104.14) (xy 138.43 111.76)
 		)
 		(stroke
@@
 	(wire
 		(pts
-			(xy 138.43 76.2) (xy 138.43 80.01)
+			(xy 123.19 99.06) (xy 130.81 99.06)
 		)
 		(stroke
@@
 	(wire
 		(pts
-			(xy 88.9 93.98) (xy 90.17 93.98)
+			(xy 138.43 76.2) (xy 138.43 80.01)
 		)
 		(stroke
@@
 	(wire
 		(pts
-			(xy 123.19 115.57) (xy 123.19 121.92)
+			(xy 88.9 93.98) (xy 90.17 93.98)
 		)
 		(stroke
@@
 	(wire
 		(pts
-			(xy 144.78 91.44) (xy 138.43 91.44)
+			(xy 123.19 115.57) (xy 123.19 121.92)
 		)
 		(stroke
@@
 	(wire
 		(pts
-			(xy 138.43 121.92) (xy 129.54 121.92)
+			(xy 138.43 111.76) (xy 138.43 121.92)
 		)
 		(stroke
@@
 	(wire
 		(pts
+			(xy 138.43 121.92) (xy 129.54 121.92)
+		)
+		(stroke
+			(width 0)
+			(type default)
+		)
+	)
+	(wire
+		(pts
 			(xy 138.43 82.55) (xy 138.43 91.44)
+		)
+		(stroke
+			(width 0)
+			(type default)
+		)
+	)
+	(wire
+		(pts
+			(xy 138.43 91.44) (xy 138.43 93.98)
 		)
 		(stroke
@@
 		)
 	)
+	(label "Mosfet_D"
+		(at 142.24 91.44 0)
+		(effects
+			(font
+				(size 1.27 1.27)
+			)
+			(justify left bottom)
+		)
+	)
 	(label "Mosfet_S"
-		(at 144.78 91.44 0)
+		(at 143.51 111.76 0)
 		(effects
 			(font
@@
 			)
 		)
-		(property "Link" "https://www.lcsc.com/product-detail/C859110.html"
-			(at 123.19 92.71 0)
-			(hide yes)
-			(show_name no)
-			(do_not_autoplace no)
-			(effects
-				(font
-					(size 1.27 1.27)
-				)
-			)
-		)
 		(property "Field7" ""
 			(at 123.19 92.71 0)
@@
 			)
 		)
-		(property "Footprint" "Package_TO_SOT_THT:TO-220-3_Horizontal_TabDown"
+		(property "Footprint" "Package_TO_SOT_THT:TO-220-3_Horizontal_TabUp"
 			(at 135.89 111.76 0)
 			(hide yes)
