File: NICROM.kicad_sch (KiCad schematic)
At the start: 6 parts, among them CN3 DB127V-5.08-2P-GN-S, Q1 IRLZ44NPBF

Commit message: VERSION FINAL
Parts:
- Q1: footprint Package_TO_SOT_THT:TO-220-3_Horizontal_TabUp -> Package_TO_SOT_THT:TO-220-3_Horizontal_TabDown
Changed lines of the file:
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@@
 			)
 		)
-		(property "Footprint" "Package_TO_SOT_THT:TO-220-3_Horizontal_TabUp"
+		(property "Footprint" "Package_TO_SOT_THT:TO-220-3_Horizontal_TabDown"
 			(at 135.89 111.76 0)
 			(hide yes)
