File: Alimentacion_V2.kicad_sch (KiCad schematic)
At the start: 18 parts, among them CN1 XT30PW-M, CN2 XT30PW-M, Q2 AOD4185_C400894, Q3 AOD4185_C400894

Commit message: 3D MODEL
Parts:
- renumbered TP11 to TP1, TP9 to TP2, TP10 to TP3, TP12 to TP4
Changed lines of the file:
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@@
 	(wire
 		(pts
-			(xy 167.64 57.15) (xy 167.64 54.61)
+			(xy 167.64 55.88) (xy 167.64 54.61)
 		)
 		(stroke
@@
 		(in_pos_files yes)
 		(dnp no)
-		(fields_autoplaced yes)
-		(property "Reference" "TP12"
+		(property "Reference" "TP4"
 			(at 215.9 50.0379 0)
 			(hide yes)
@@
 		)
 		(property "Description" "GND"
-			(at 213.36 54.61 0)
+			(at 213.36 48.768 0)
 			(show_name no)
 			(do_not_autoplace no)
@@
 			(project "ARLISS_STM32_2026"
 				(path "/9719ea46-14c4-4409-9c57-49dd5454c03f/efeb48d2-be8c-4c47-a263-81c8c7c61051"
-					(reference "TP12")
+					(reference "TP4")
 					(unit 1)
 				)
@@
 	(symbol
 		(lib_id "power:+3.3V")
-		(at 167.64 57.15 0)
+		(at 167.64 55.88 0)
 		(mirror x)
 		(unit 1)
@@
 		(fields_autoplaced yes)
 		(property "Reference" "#PWR0179"
-			(at 167.64 53.34 0)
+			(at 167.64 52.07 0)
 			(hide yes)
 			(show_name no)
@@
 		)
 		(property "Value" "+3.3V"
-			(at 167.64 62.23 0)
+			(at 167.64 60.96 0)
 			(show_name no)
 			(do_not_autoplace no)
@@
 		)
 		(property "Footprint" ""
-			(at 167.64 57.15 0)
+			(at 167.64 55.88 0)
 			(hide yes)
 			(show_name no)
@@
 		)
 		(property "Datasheet" ""
-			(at 167.64 57.15 0)
-			(hide yes)
-			(show_name no)
-			(do_not_autoplace no)
-			(effects
-				(font
-					(size 1.27 1.27)
-				)
-			)
-		)
-		(property "Description" "Power symbol creates a global label with name \"+3.3V\""
-			(at 167.64 57.15 0)
-			(hide yes)
+			(at 167.64 55.88 0)
+			(hide yes)
+			(show_name no)
+			(do_not_autoplace no)
+			(effects
+				(font
+					(size 1.27 1.27)
+				)
+			)
+		)
+		(property "Description" "3V3"
+			(at 167.64 55.88 0)
 			(show_name no)
 			(do_not_autoplace no)
@@
 		(in_pos_files yes)
 		(dnp no)
-		(fields_autoplaced yes)
-		(property "Reference" "TP10"
+		(property "Reference" "TP3"
 			(at 198.12 50.0379 0)
+			(hide yes)
 			(show_name no)
 			(do_not_autoplace no)
@@
 		)
 		(property "Description" "GND"
-			(at 195.58 54.61 0)
-			(hide yes)
+			(at 195.58 48.768 0)
 			(show_name no)
 			(do_not_autoplace no)
@@
 			(project "ARLISS_STM32_2026"
 				(path "/9719ea46-14c4-4409-9c57-49dd5454c03f/efeb48d2-be8c-4c47-a263-81c8c7c61051"
-					(reference "TP10")
+					(reference "TP3")
 					(unit 1)
 				)
@@
 		(in_pos_files yes)
 		(dnp no)
-		(fields_autoplaced yes)
-		(property "Reference" "TP9"
+		(property "Reference" "TP2"
 			(at 182.88 52.5781 0)
+			(hide yes)
 			(show_name no)
 			(do_not_autoplace no)
@@
 		)
 		(property "Description" "11.1V"
-			(at 180.34 54.61 0)
+			(at 180.34 48.26 0)
 			(show_name no)
 			(do_not_autoplace no)
@@
 			(project "ARLISS_STM32_2026"
 				(path "/9719ea46-14c4-4409-9c57-49dd5454c03f/efeb48d2-be8c-4c47-a263-81c8c7c61051"
-					(reference "TP9")
+					(reference "TP2")
 					(unit 1)
 				)
@@
 		(in_pos_files yes)
 		(dnp no)
-		(property "Reference" "TP11"
+		(property "Reference" "TP1"
 			(at 170.434 48.514 0)
+			(hide yes)
 			(show_name no)
 			(do_not_autoplace no)
@@
 		)
 		(property "Value" "TestPoint"
-			(at 170.434 45.974 0)
+			(at 172.212 48.768 0)
 			(show_name no)
 			(do_not_autoplace no)
@@
 			(project "ARLISS_STM32_2026"
 				(path "/9719ea46-14c4-4409-9c57-49dd5454c03f/efeb48d2-be8c-4c47-a263-81c8c7c61051"
-					(reference "TP11")
+					(reference "TP1")
 					(unit 1)
 				)

Commit message: Primer_plano
Connections:
- net +BATT1: now also F1.2; no longer F2.2
- net +BATT2: now also F2.2; no longer F1.2
- net at F2.1: now also Q2.2 (D); no longer Q3.2 (D)
- net at F1.1: now also Q3.2 (D); no longer Q2.2 (D)
Changed lines of the file:
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@@
 	(text "BATT_11.1V"
 		(exclude_from_sim no)
-		(at 54.61 94.234 0)
+		(at 55.118 58.42 0)
 		(effects
 			(font
@@
 	(text "BATT_7.4V"
 		(exclude_from_sim no)
-		(at 55.118 56.642 0)
+		(at 56.642 94.996 0)
 		(effects
 			(font
@@
 			(width 0)
 			(type default)
+		)
+	)
+	(symbol
+		(lib_id "CANSAT_STM32_symbols:0466.750NRHF")
+		(at 124.46 102.87 90)
+		(unit 1)
+		(body_style 1)
+		(exclude_from_sim no)
+		(in_bom yes)
+		(on_board yes)
+		(in_pos_files yes)
+		(dnp no)
+		(fields_autoplaced yes)
+		(property "Reference" "F2"
+			(at 127 101.5999 90)
+			(show_name no)
+			(do_not_autoplace no)
+			(effects
+				(font
+					(size 1.27 1.27)
+				)
+				(justify right)
+			)
+		)
+		(property "Value" "750mA"
+			(at 127 104.1399 90)
+			(show_name no)
+			(do_not_autoplace no)
+			(effects
+				(font
+					(size 1.27 1.27)
+				)
+				(justify right)
+			)
+		)
+		(property "Footprint" "ARLISS-footprints:F1206"
+			(at 132.08 102.87 0)
+			(hide yes)
+			(show_name no)
+			(do_not_autoplace no)
+			(effects
+				(font
+					(size 1.27 1.27)
+				)
+			)
+		)
+		(property "Datasheet" "https://lcsc.com/product-detail/Blade-Fuses_Littelfuse_0466-750NRHF_Littelfuse-0466-750NRHF_C187594.html"
+			(at 134.62 102.87 0)
+			(hide yes)
+			(show_name no)
+			(do_not_autoplace no)
+			(effects
+				(font
+					(size 1.27 1.27)
+				)
+			)
+		)
+		(property "Description" ""
+			(at 124.46 102.87 0)
+			(hide yes)
+			(show_name no)
+			(do_not_autoplace no)
+			(effects
+				(font
+					(size 1.27 1.27)
+				)
+			)
+		)
+		(property "Manufacturer" "Littelfuse(美国力特)"
+			(at 137.16 102.87 0)
+			(hide yes)
+			(show_name no)
+			(do_not_autoplace no)
+			(effects
+				(font
+					(size 1.27 1.27)
+				)
+			)
+		)
+		(property "MPN" "0466.750NRHF"
+			(at 139.7 102.87 0)
+			(hide yes)
+			(show_name no)
+			(do_not_autoplace no)
+			(effects
+				(font
+					(size 1.27 1.27)
+				)
+			)
+		)
+		(property "LCSC Part" "C187594"
+			(at 142.24 102.87 0)
+			(hide yes)
+			(show_name no)
+			(do_not_autoplace no)
+			(effects
+				(font
+					(size 1.27 1.27)
+				)
+			)
+		)
+		(pin "1"
+		)
+		(pin "2"
+		)
+		(instances
+			(project "ARLISS_STM32_2026"
+				(path "/9719ea46-14c4-4409-9c57-49dd5454c03f/efeb48d2-be8c-4c47-a263-81c8c7c61051"
+					(reference "F2")
+					(unit 1)
+				)
+			)
 		)
 	)
@@
 	)
 	(symbol
-		(lib_id "CANSAT_STM32_symbols:0466.750NRHF")
-		(at 123.19 54.61 90)
-		(unit 1)
-		(body_style 1)
-		(exclude_from_sim no)
-		(in_bom yes)
-		(on_board yes)
-		(in_pos_files yes)
-		(dnp no)
-		(fields_autoplaced yes)
-		(property "Reference" "F2"
-			(at 125.73 53.3399 90)
-			(show_name no)
-			(do_not_autoplace no)
-			(effects
-				(font
-					(size 1.27 1.27)
-				)
-				(justify right)
-			)
-		)
-		(property "Value" "750mA"
-			(at 125.73 55.8799 90)
-			(show_name no)
-			(do_not_autoplace no)
-			(effects
-				(font
-					(size 1.27 1.27)
-				)
-				(justify right)
-			)
-		)
-		(property "Footprint" "ARLISS-footprints:F1206"
-			(at 130.81 54.61 0)
-			(hide yes)
-			(show_name no)
-			(do_not_autoplace no)
-			(effects
-				(font
-					(size 1.27 1.27)
-				)
-			)
-		)
-		(property "Datasheet" "https://lcsc.com/product-detail/Blade-Fuses_Littelfuse_0466-750NRHF_Littelfuse-0466-750NRHF_C187594.html"
-			(at 133.35 54.61 0)
-			(hide yes)
-			(show_name no)
-			(do_not_autoplace no)
-			(effects
-				(font
-					(size 1.27 1.27)
-				)
-			)
-		)
-		(property "Description" ""
-			(at 123.19 54.61 0)
-			(hide yes)
-			(show_name no)
-			(do_not_autoplace no)
-			(effects
-				(font
-					(size 1.27 1.27)
-				)
-			)
-		)
-		(property "Manufacturer" "Littelfuse(美国力特)"
-			(at 135.89 54.61 0)
-			(hide yes)
-			(show_name no)
-			(do_not_autoplace no)
-			(effects
-				(font
-					(size 1.27 1.27)
-				)
-			)
-		)
-		(property "MPN" "0466.750NRHF"
-			(at 138.43 54.61 0)
-			(hide yes)
-			(show_name no)
-			(do_not_autoplace no)
-			(effects
-				(font
-					(size 1.27 1.27)
-				)
-			)
-		)
-		(property "LCSC Part" "C187594"
-			(at 140.97 54.61 0)
-			(hide yes)
-			(show_name no)
-			(do_not_autoplace no)
-			(effects
-				(font
-					(size 1.27 1.27)
-				)
-			)
-		)
-		(pin "1"
-		)
-		(pin "2"
-		)
-		(instances
-			(project "ARLISS_STM32_2026"
-				(path "/9719ea46-14c4-4409-9c57-49dd5454c03f/efeb48d2-be8c-4c47-a263-81c8c7c61051"
-					(reference "F2")
-					(unit 1)
-				)
-			)
-		)
-	)
-	(symbol
 		(lib_id "power:+BATT")
 		(at 124.46 123.19 270)
@@
 	)
 	(symbol
+		(lib_id "CANSAT_STM32_symbols:LTC1206-1700TS")
+		(at 123.19 54.61 90)
+		(unit 1)
+		(body_style 1)
+		(exclude_from_sim no)
+		(in_bom yes)
+		(on_board yes)
+		(in_pos_files yes)
+		(dnp no)
+		(fields_autoplaced yes)
+		(property "Reference" "F1"
+			(at 125.73 53.3399 90)
+			(show_name no)
+			(do_not_autoplace no)
+			(effects
+				(font
+					(size 1.27 1.27)
+				)
+				(justify right)
+			)
+		)
+		(property "Value" "7A"
+			(at 125.73 55.8799 90)
+			(show_name no)
+			(do_not_autoplace no)
+			(effects
+				(font
+					(size 1.27 1.27)
+				)
+				(justify right)
+			)
+		)
+		(property "Footprint" "ARLISS-footprints:F1206"
+			(at 130.81 54.61 0)
+			(hide yes)
+			(show_name no)
+			(do_not_autoplace no)
+			(effects
+				(font
+					(size 1.27 1.27)
+				)
+			)
+		)
+		(property "Datasheet" "https://www.lcsc.com/datasheet/C52988555.pdf"
+			(at 133.35 54.61 0)
+			(hide yes)
+			(show_name no)
+			(do_not_autoplace no)
+			(effects
+				(font
+					(size 1.27 1.27)
+				)
+			)
+		)
+		(property "Description" ""
+			(at 123.19 54.61 0)
+			(hide yes)
+			(show_name no)
+			(do_not_autoplace no)
+			(effects
+				(font
+					(size 1.27 1.27)
+				)
+			)
+		)
+		(property "Manufacturer" "LUTE(陆特)"
+			(at 135.89 54.61 0)
+			(hide yes)
+			(show_name no)
+			(do_not_autoplace no)
+			(effects
+				(font
+					(size 1.27 1.27)
+				)
+			)
+		)
+		(property "MPN" "LTC1206-1700TS"
+			(at 138.43 54.61 0)
+			(hide yes)
+			(show_name no)
+			(do_not_autoplace no)
+			(effects
+				(font
+					(size 1.27 1.27)
+				)
+			)
+		)
+		(property "LCSC Part" "C52988555"
+			(at 140.97 54.61 0)
+			(hide yes)
+			(show_name no)
+			(do_not_autoplace no)
+			(effects
+				(font
+					(size 1.27 1.27)
+				)
+			)
+		)
+		(pin "2"
+		)
+		(pin "1"
+		)
+		(instances
+			(project "ARLISS_STM32_2026"
+				(path "/9719ea46-14c4-4409-9c57-49dd5454c03f/efeb48d2-be8c-4c47-a263-81c8c7c61051"
+					(reference "F1")
+					(unit 1)
+				)
+			)
+		)
+	)
+	(symbol
 		(lib_id "Device:D_Zener")
 		(at 115.57 76.2 180)
@@
 					(unit 1)
 				)
-			)
-		)
-	)
-	(symbol
-		(lib_id "CANSAT_STM32_symbols:LTC1206-1700TS")
-		(at 124.46 102.87 90)
-		(unit 1)
-		(body_style 1)
-		(exclude_from_sim no)
-		(in_bom yes)
-		(on_board yes)
-		(in_pos_files yes)
-		(dnp no)
-		(fields_autoplaced yes)
-		(property "Reference" "F1"
-			(at 127 101.5999 90)
-			(show_name no)
-			(do_not_autoplace no)
-			(effects
-				(font
-					(size 1.27 1.27)
-				)
-				(justify right)
-			)
-		)
-		(property "Value" "7A"
-			(at 127 104.1399 90)
-			(show_name no)
-			(do_not_autoplace no)
-			(effects
-				(font
-					(size 1.27 1.27)
-				)
-				(justify right)
-			)
-		)
-		(property "Footprint" "ARLISS-footprints:F1206"
-			(at 132.08 102.87 0)
-			(hide yes)
-			(show_name no)
-			(do_not_autoplace no)
-			(effects
-				(font
-					(size 1.27 1.27)
-				)
-			)
-		)
-		(property "Datasheet" "https://www.lcsc.com/datasheet/C52988555.pdf"
-			(at 134.62 102.87 0)
-			(hide yes)
-			(show_name no)
-			(do_not_autoplace no)
-			(effects
-				(font
-					(size 1.27 1.27)
-				)
-			)
-		)
-		(property "Description" ""
-			(at 124.46 102.87 0)
-			(hide yes)
-			(show_name no)
-			(do_not_autoplace no)
-			(effects
-				(font
-					(size 1.27 1.27)
-				)
-			)
-		)
-		(property "Manufacturer" "LUTE(陆特)"
-			(at 137.16 102.87 0)
-			(hide yes)
-			(show_name no)
-			(do_not_autoplace no)
-			(effects
-				(font
-					(size 1.27 1.27)
-				)
-			)
-		)
-		(property "MPN" "LTC1206-1700TS"
-			(at 139.7 102.87 0)
-			(hide yes)
-			(show_name no)
-			(do_not_autoplace no)
-			(effects
-				(font
-					(size 1.27 1.27)
-				)
-			)
-		)
-		(property "LCSC Part" "C52988555"
-			(at 142.24 102.87 0)
-			(hide yes)
-			(show_name no)
-			(do_not_autoplace no)
-			(effects
-				(font
-					(size 1.27 1.27)
-				)
-			)
-		)
-		(pin "2"
-		)
-		(pin "1"
-		)
-		(instances
-			(project "ARLISS_STM32_2026"
-				(path "/9719ea46-14c4-4409-9c57-49dd5454c03f/efeb48d2-be8c-4c47-a263-81c8c7c61051"
-					(reference "F1")
-					(unit 1)
-				)

Commit message: V3
Parts:
- added C2: 100nF, Capacitor_SMD:C_0603_1608Metric_Pad1.08x0.95mm_HandSolder, symbol CANSAT_STM32_symbols:TCC0402X7R104J500AT
- added C33: 10uF, Capacitor_SMD:C_0805_2012Metric_Pad1.18x1.45mm_HandSolder, symbol CANSAT_STM32_symbols:CL21B106KAYQNNE
- added C34, C35: 22uF, Capacitor_SMD:C_0805_2012Metric_Pad1.18x1.45mm_HandSolder, symbol CANSAT_STM32_symbols:TCC0402X7R104J500AT
- added L2: 3.3uH, ARLISS-footprints:IND-SMD_L4.1-W4.1_FTC404020S, symbol CANSAT_STM32_symbols:FTC404020S3R3MGCA
- added U7: AP63203QWU-7, ARLISS-footprints:TSOT-26_L2.9-W1.6-P0.95-LS2.8-BL, symbol CANSAT_STM32_symbols:AP63203QWU-7
Connections:
- net +3.3V: now also C34.2, C35.2, L2.2, U7.1 (FB)
- net GND: now also C33.1, C34.1, C35.1, U7.4 (GND)
- new net: C2.1, L2.1, U7.5 (SW)
- new net: C2.2, U7.6 (BST)
- new net: C33.2, U7.2 (EN), U7.3 (VIN)

Commit message: REV_1
Connections:
- net +VDC: now reaches C33.2, U7.2 (EN), U7.3 (VIN)

Commit message: VERSION FINAL
Parts:
- F2: LCSC Part C187594 -> C83557; MPN 0466.750NRHF -> 0466.250NRHF
